File: PCB/STEVEannouncer.kicad_pcb (KiCad board)
At the start: 2 copper layers, 31 parts, among them J1 Barrel_Jack, J2 NC3FAH, J3 XLR3_Ground, J4 NC3MAH, J5 NC3MAH, J7 AudioJack3_Dual_Ground_Switch, SW1 SW_SPST, U2 TMUX6236, U4 THAT1646, U5 THAT1646, U6 OPA1678, U7 OPA1622, U8 LV3842, U9 LV3842

Commit message: Wooooooo
Parts:
- removed D8: BAS716, Diode_SMD:D_SOD-523
- removed J1: Barrel_Jack, Connector_BarrelJack:BarrelJack_Horizontal
- removed J7: AudioJack3_Dual_Ground_Switch, Connector_Audio:Jack_6.35mm_Neutrik_NSJ12HF-1_Horizontal
- removed U4: THAT1646, Package_SO:SO-8_3.9x4.9mm_P1.27mm
- added C201: 1u/50V, Capacitor_SMD:C_0402_1005Metric, F.Cu at (66.4, 44.5)
- added C202: 1000u, Capacitor_SMD:CP_Elec_16x17.5, F.Cu at (59.3, 34.5)
- added C203: 2.2u, Capacitor_SMD:C_0603_1608Metric, F.Cu at (69.9, 44.8)
- added C204: 2.2u, Capacitor_SMD:C_0603_1608Metric, F.Cu at (69.9, 47.3)
- added C205: 100n, Capacitor_SMD:C_0402_1005Metric, F.Cu at (66.4, 46.5)
- added C206: 100n, Capacitor_SMD:C_0402_1005Metric, F.Cu at (66.4, 48.5)
- added C207: 22u, Capacitor_SMD:C_1206_3216Metric, F.Cu at (56.0, 45.2)
- added C208: 22u, Capacitor_SMD:C_1206_3216Metric, F.Cu at (56.0, 48.6)
- added C301: 100p, Capacitor_SMD:C_0402_1005Metric, F.Cu at (60.0, 2.49)
- added C302: 470p, Capacitor_SMD:C_0402_1005Metric, F.Cu at (60.0, 4.46)
- added C303: 470p, Capacitor_SMD:C_0402_1005Metric, F.Cu at (60.0, 6.43)
- added C304: 22u, Capacitor_SMD:CP_Elec_6.3x7.7, F.Cu at (63.8, -10.7)
- added C305: 22u, Capacitor_SMD:CP_Elec_6.3x7.7, F.Cu at (63.8, -2.57)
- added C306: 100u, Capacitor_SMD:C_1206_3216Metric, F.Cu at (69.8, 15.6)
- added C307: 100n, Capacitor_SMD:C_0402_1005Metric, F.Cu at (60.0, 8.40)
- added C308: 100n, Capacitor_SMD:C_0402_1005Metric, F.Cu at (62.8, 2.49)
- added C309: 100n, Capacitor_SMD:C_0402_1005Metric, F.Cu at (62.8, 4.46)
- added C310: 100n, Capacitor_SMD:C_0402_1005Metric, F.Cu at (62.8, 6.43)
- added C311: 100n, Capacitor_SMD:C_0402_1005Metric, F.Cu at (62.8, 8.40)
- added C312: 100n, Capacitor_SMD:C_0402_1005Metric, F.Cu at (65.7, 2.49)
- added C313: 100n, Capacitor_SMD:C_0402_1005Metric, F.Cu at (65.7, 4.46)
- added C314: 100n, Capacitor_SMD:C_0402_1005Metric, F.Cu at (65.7, 6.43)
- added C315: 100n, Capacitor_SMD:C_0402_1005Metric, F.Cu at (65.7, 8.40)
- added C316: 10u, Capacitor_SMD:C_0603_1608Metric, F.Cu at (69.0, 18.5)
- added C317: 10u, Capacitor_SMD:C_0603_1608Metric, F.Cu at (69.0, 21.1)
- added C318: 100p, Capacitor_SMD:C_0402_1005Metric, F.Cu at (68.6, 2.49)
- added C319: 100p, Capacitor_SMD:C_0402_1005Metric, F.Cu at (68.6, 4.46)
- added C320: 100p, Capacitor_SMD:C_0402_1005Metric, F.Cu at (68.6, 6.43)
- added C321: 100p, Capacitor_SMD:C_0402_1005Metric, F.Cu at (68.6, 8.40)
- added C401: 1u/50V, Capacitor_SMD:C_0402_1005Metric, F.Cu at (25.9, 21.8)
- added C402: 1u/50V, Capacitor_SMD:C_0402_1005Metric, F.Cu at (25.9, 23.8)
- added C403: 100p, Capacitor_SMD:C_0402_1005Metric, F.Cu at (25.9, 25.7)
- added C404: 100p, Capacitor_SMD:C_0402_1005Metric, F.Cu at (25.9, 27.7)
- added C405: 100n, Capacitor_SMD:C_0402_1005Metric, F.Cu at (25.9, 29.7)
- added C406: 100n, Capacitor_SMD:C_0402_1005Metric, F.Cu at (25.9, 31.6)
- added C407: 1u/50V, Capacitor_SMD:C_0402_1005Metric, F.Cu at (28.8, 21.8)
- added C408: 100p, Capacitor_SMD:C_0402_1005Metric, F.Cu at (28.8, 23.8)
- added C409: 100p, Capacitor_SMD:C_0402_1005Metric, F.Cu at (28.8, 25.7)
- added C410: 100n, Capacitor_SMD:C_0402_1005Metric, F.Cu at (28.8, 27.7)
- added C411: 100n, Capacitor_SMD:C_0402_1005Metric, F.Cu at (28.8, 29.7)
- added C412: 100n, Capacitor_SMD:C_0402_1005Metric, F.Cu at (28.8, 31.6)
- added C413: 100n, Capacitor_SMD:C_0402_1005Metric, F.Cu at (31.6, 21.8)
- added C414: 100n, Capacitor_SMD:C_0402_1005Metric, F.Cu at (31.6, 23.8)
- added C415: 100n, Capacitor_SMD:C_0402_1005Metric, F.Cu at (31.6, 25.7)
- added D202: D_Schottky, Diode_SMD:D_SOD-523, F.Cu at (69.7, 49.8)
- added D203: D_Schottky, Diode_SMD:D_SOD-523, F.Cu at (69.7, 52.2)
- added D308: BAS716, Diode_SMD:D_SOD-523, F.Cu at (72.8, 18.5)
- added D406: BAS716, Diode_SMD:D_SOD-523, F.Cu at (9.02, 24.6)
- added J202: Barrel_Jack_Switch, STEVEannouncer:Barrel Jack, F.Cu at (178.1, 88.9)
- added J302: Conn_01x02, Connector_JST:JST_PH_B2B-PH-SM4-TB_1x02-1MP_P2.00mm_Vertical, F.Cu at (53.3, -9.52)
- added J303: Conn_01x02, Connector_JST:JST_PH_B2B-PH-SM4-TB_1x02-1MP_P2.00mm_Vertical, F.Cu at (53.3, 0.03)
- added J304: Conn_01x02, Connector_JST:JST_PH_B2B-PH-SM4-TB_1x02-1MP_P2.00mm_Vertical, F.Cu at (53.3, 9.58)
- added J305: Conn_01x02, Connector_JST:JST_PH_B2B-PH-SM4-TB_1x02-1MP_P2.00mm_Vertical, F.Cu at (53.3, 19.1)
- added J402: Conn_01x03, Connector_JST:JST_PH_B3B-PH-SM4-TB_1x03-1MP_P2.00mm_Vertical, F.Cu at (4.60, -9.52)
- added J403: Conn_01x03, Connector_JST:JST_PH_B3B-PH-SM4-TB_1x03-1MP_P2.00mm_Vertical, F.Cu at (4.60, 0.03)
- added J404: Conn_01x03, Connector_JST:JST_PH_B3B-PH-SM4-TB_1x03-1MP_P2.00mm_Vertical, F.Cu at (4.60, 9.58)
- added J405: Conn_01x03, Connector_JST:JST_PH_B3B-PH-SM4-TB_1x03-1MP_P2.00mm_Vertical, F.Cu at (4.60, 19.1)
- added J406: NRJ6HF, Connector_Audio:Jack_6.35mm_Neutrik_NRJ6HF_Horizontal, F.Cu at (152.9, 132.8)
- added J407: NRJ6HF, Connector_Audio:Jack_6.35mm_Neutrik_NRJ6HF_Horizontal, F.Cu at (135.1, 132.8)
- added L201: 18u, STEVEannouncer:Inductor 3012, F.Cu at (50.6, 46.1)
- added L202: 18u, STEVEannouncer:Inductor 3012, F.Cu at (50.6, 51.2)
- added Q201: BC847, Package_TO_SOT_SMD:SOT-523, F.Cu at (55.1, 51.8)
- added Q202: BCV49, Package_TO_SOT_SMD:SOT-89-3, F.Cu at (62.2, 46.7)
- added R201: 1Meg, Resistor_SMD:R_0402_1005Metric, F.Cu at (71.7, 26.4)
- added R202: 330k, Resistor_SMD:R_0402_1005Metric, F.Cu at (71.7, 28.4)
- added R203: 20k, Resistor_SMD:R_0402_1005Metric, F.Cu at (71.7, 30.4)
- added R205: 10, Resistor_SMD:R_1206_3216Metric, F.Cu at (61.6, 51.3)
- added R206: 20k, Resistor_SMD:R_0402_1005Metric, F.Cu at (71.7, 32.4)
- added R207: 20k, Resistor_SMD:R_0402_1005Metric, F.Cu at (71.7, 34.4)
- added R208: 80.6k, Resistor_SMD:R_0402_1005Metric, F.Cu at (71.7, 36.4)
- added R209: 80.6k, Resistor_SMD:R_0402_1005Metric, F.Cu at (71.7, 38.3)
- added R301: 10, Resistor_SMD:R_1206_3216Metric, F.Cu at (61.3, 17.6)
- added R302: 10, Resistor_SMD:R_1206_3216Metric, F.Cu at (61.3, 20.9)
- added R303: 1k, Resistor_SMD:R_0402_1005Metric, F.Cu at (70.4, -13.8)
- added R304: 1k, Resistor_SMD:R_0402_1005Metric, F.Cu at (70.4, -11.8)
- added R305: 20k, Resistor_SMD:R_0402_1005Metric, F.Cu at (70.4, -9.82)
- added R306: 270, Resistor_SMD:R_0402_1005Metric, F.Cu at (70.4, -7.83)
- added R307: 20k, Resistor_SMD:R_0402_1005Metric, F.Cu at (70.4, -5.84)
- added R308: 20k, Resistor_SMD:R_0402_1005Metric, F.Cu at (70.4, -3.85)
- added R309: 20k, Resistor_SMD:R_0402_1005Metric, F.Cu at (70.4, -1.86)
- added R310: 1k, Resistor_SMD:R_0402_1005Metric, F.Cu at (73.3, -13.8)
- added R311: 100, Resistor_SMD:R_0402_1005Metric, F.Cu at (73.3, -11.8)
- added R312: 1k, Resistor_SMD:R_0402_1005Metric, F.Cu at (73.3, -9.82)
- added R313: 20k, Resistor_SMD:R_0402_1005Metric, F.Cu at (73.3, -7.83)
- added R314: 10k, Resistor_SMD:R_0402_1005Metric, F.Cu at (73.3, -5.84)
- added R315: 20k, Resistor_SMD:R_0402_1005Metric, F.Cu at (73.3, -3.85)
- added R316: 1k, Resistor_SMD:R_0402_1005Metric, F.Cu at (73.3, -1.86)
- added R317: 1k, Resistor_SMD:R_0402_1005Metric, F.Cu at (76.2, -13.8)
- added R318: 100, Resistor_SMD:R_0402_1005Metric, F.Cu at (76.2, -11.8)
- added R319: 20k, Resistor_SMD:R_0402_1005Metric, F.Cu at (76.2, -9.82)
- added R320: 20k, Resistor_SMD:R_0402_1005Metric, F.Cu at (76.2, -7.83)
- added R401: 20k, Resistor_SMD:R_0402_1005Metric, F.Cu at (34.5, 21.8)
- added R402: 20k, Resistor_SMD:R_0402_1005Metric, F.Cu at (34.5, 23.8)
- added R403: 6.8k, Resistor_SMD:R_0402_1005Metric, F.Cu at (34.5, 25.8)
- added R404: 6.8k, Resistor_SMD:R_0402_1005Metric, F.Cu at (34.5, 27.8)
- added R405: 80.6k, Resistor_SMD:R_0402_1005Metric, F.Cu at (34.5, 29.8)
- added R406: 80.6k, Resistor_SMD:R_0402_1005Metric, F.Cu at (37.5, 21.8)
- added R407: 80.6k, Resistor_SMD:R_0402_1005Metric, F.Cu at (37.5, 23.8)
- added R408: 20k, Resistor_SMD:R_0402_1005Metric, F.Cu at (37.5, 25.8)
- added R409: 20k, Resistor_SMD:R_0402_1005Metric, F.Cu at (37.5, 27.8)
- added R410: 1Meg, Resistor_SMD:R_0402_1005Metric, F.Cu at (37.5, 29.8)
- added R411: 10k, Resistor_SMD:R_0402_1005Metric, F.Cu at (40.4, 21.8)
- added R412: 330k, Resistor_SMD:R_0402_1005Metric, F.Cu at (40.4, 23.8)
- added R413: 330k, Resistor_SMD:R_0402_1005Metric, F.Cu at (40.4, 25.8)
- added RV401: 10k, STEVEannouncer:Pot, F.Cu at (234.3, 69.9)
- added RV402: 10k, STEVEannouncer:Pot, F.Cu at (234.6, 79.8)
- added SW302: SW_SPST, Button_Switch_Keyboard:SW_Cherry_MX_1.00u_PCB, F.Cu at (236.7, 95.6)
- added U301: THAT1512, Package_SO:SO-8_3.9x4.9mm_P1.27mm, F.Cu at (62.8, 12.7)
- added U303: OPA1678, Package_SON:WSON-8-1EP_3x3mm_P0.5mm_EP1.2x2mm_ThermalVias, F.Cu at (70.1, 11.7)
- added U401: THAT2162, Package_SO:QSOP-16_3.9x4.9mm_P0.635mm, F.Cu at (2.98, 26.6)
- J401: renamed from J3; value XLR3_Ground -> ~
- U403: renamed from U7; footprint Package_SON:Texas_S-PVSON-N10 -> Package_SON:Texas_S-PVSON-N10_ThermalVias
- moved SW301 139.4 mm to (237.3, 119.0)
- moved J301 73.1 mm to (107.0, 139.3), turned to -90 degrees
- renumbered D13 to D201, D1 to D301, D6 to D302, D7 to D303, D4 to D304, D5 to D305, D2 to D306, D3 to D307, D9 to D401, D11 to D402, D10 to D403, D12 to D404, FB1 to FB301, FB2 to FB302, FB3 to FB303, FB4 to FB304, J2 to J301, J5 to J306, J4 to J307, SW1 to SW301, U8 to U201, U9 to U202, U2 to U302, U5 to U304, U6 to U402
Connections:
- SW301 pad 1: Net-(SW1-A) -> Net-(J303-Pin_1)
- SW301 pad 2: +5V -> Net-(J303-Pin_2)
- U302 pad 1: Net-(SW1-A) -> Net-(D308-K)
- U302 pad 10: Net-(U2B-SA) -> Net-(U301-Out)
- U302 pad 11: Net-(U2A-SB) -> Net-(U302B-D)
- U302 pad 12: Net-(U2B-SB) -> GND
- U302 pad 15: (no net) -> unconnected-(U302C-NC-Pad15)
- U302 pad 16: (no net) -> unconnected-(U302C-NC-Pad16)
- U302 pad 2: unconnected-(U2A-SA-Pad2) -> GND
- U302 pad 3: Net-(U1-Out) -> Net-(U302A-D)
- U302 pad 4: Net-(U2A-SB) -> Net-(U301-Out)
- U302 pad 6: (no net) -> GND
- U302 pad 7: (no net) -> unconnected-(U302C-NC-Pad7)
- U302 pad 8: (no net) -> unconnected-(U302C-NC-Pad8)
- U304 pad 4: Net-(U2B-SB) -> Net-(U302A-D)
- U402 pad 4: +5V -> -5V
- U402 pad 8: -5V -> +5V
- U402 pad 9: (no net) -> -5V
- U403 pad 8: +5V -> Net-(D406-A)

Commit message: lalalalala
Parts:
- removed D406: BAS716, Diode_SMD:D_SOD-523
- removed J202: Barrel_Jack_Switch, STEVEannouncer:Barrel Jack
- removed R209: 80.6k, Resistor_SMD:R_0402_1005Metric
- added D405: BAS716, Diode_SMD:D_SOD-523, F.Cu at (135.0, 126.0)
- added H101: MountingHole, MountingHole:MountingHole_3.2mm_M3, F.Cu at (91.0, 136.0)
- added H102: MountingHole, MountingHole:MountingHole_3.2mm_M3, F.Cu at (91.0, 75.0)
- added H103: MountingHole, MountingHole:MountingHole_3.2mm_M3, F.Cu at (189.0, 136.0)
- added H104: MountingHole, MountingHole:MountingHole_3.2mm_M3, F.Cu at (189.0, 75.0)
- added J201: Barrel_Jack_Switch, STEVEannouncer:Barrel Jack, F.Cu at (179.0, 72.9)
- added R204: 10, Resistor_SMD:R_1206_3216Metric, F.Cu at (190.0, 99.0)
- C301: value 100p -> 100n
- C302: value 470p -> 100p
- C304: value 22u -> 470p; footprint Capacitor_SMD:CP_Elec_6.3x7.7 -> Capacitor_SMD:C_0402_1005Metric
- C306: value 100u -> 22u; footprint Capacitor_SMD:C_1206_3216Metric -> Capacitor_SMD:CP_Elec_6.3x7.7
- C307: value 100n -> 100u; footprint Capacitor_SMD:C_0402_1005Metric -> Capacitor_SMD:C_1206_3216Metric
- C407: value 1u/50V -> 100p
- C409: value 100p -> 1u/50V
- D302, D303: value BAS716 -> DFLZ5V6; footprint Diode_SMD:D_SOD-523 -> Diode_SMD:D_PowerDI-123
- D304, D305: value DFLZ5V6 -> BAS716; footprint Diode_SMD:D_PowerDI-123 -> Diode_SMD:D_SOD-523
- D306: value BAS3007ARPPE6327HTSA1 -> BAS716; footprint Package_TO_SOT_SMD:SOT-143 -> Diode_SMD:D_SOD-523
- D308: value BAS716 -> BAS3007ARPPE6327HTSA1; footprint Diode_SMD:D_SOD-523 -> Package_TO_SOT_SMD:SOT-143
- R205: value 10 -> 20k; footprint Resistor_SMD:R_1206_3216Metric -> Resistor_SMD:R_0402_1005Metric
- R207, R408, R409: value 20k -> 80.6k
- R307, R308, R309: value 20k -> 330k
- R310: value 1k -> 330k
- R311: value 100 -> 20k
- R312: value 1k -> 10k
- R314, R411: value 10k -> 20k
- R315: value 20k -> 1k
- R318: value 100 -> 1k
- R319, R320: value 20k -> 100
- R405, R406: value 80.6k -> 330k
- R410: value 1Meg -> 10k
- R412: value 330k -> 20k
- R413: value 330k -> 1Meg
- U301: value THAT1512 -> TMUX6236; footprint Package_SO:SO-8_3.9x4.9mm_P1.27mm -> Package_SO:TSSOP-16_4.4x5mm_P0.65mm
- U302: value TMUX6236 -> OPA1678; footprint Package_SO:TSSOP-16_4.4x5mm_P0.65mm -> Package_SON:WSON-8-1EP_3x3mm_P0.5mm_EP1.2x2mm_ThermalVias
- U303: value OPA1678 -> THAT1512; footprint Package_SON:WSON-8-1EP_3x3mm_P0.5mm_EP1.2x2mm_ThermalVias -> Package_SO:SO-8_3.9x4.9mm_P1.27mm
- moved J305 227.3 mm to (253.0, 127.7)
- moved J302 227.3 mm to (253.0, 99.0)
- moved J403 208.0 mm to (163.0, 134.9)
- moved J405 201.7 mm to (163.0, 144.0)
- moved C405 184.6 mm to (173.1, 141.0)
- moved C406 184.6 mm to (173.1, 143.0)
- moved C412 184.6 mm to (176.0, 143.0)
- moved C413 183.6 mm to (173.0, 139.0)
- moved R405 179.3 mm to (176.0, 140.0)
- moved R406 179.3 mm to (178.9, 132.0)
- moved R407 179.3 mm to (178.9, 134.0)
- moved R408 179.3 mm to (178.9, 136.0)
- moved R409 179.3 mm to (178.9, 138.0)
- moved R410 179.3 mm to (178.9, 140.0)
- moved U402 175.8 mm to (174.0, 136.0)
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Connections:
- C301 pad 1: GND -> -5V
- C301 pad 2: Net-(C301-Pad2) -> +5V
- C302 pad 1: Net-(C302-Pad1) -> GND
- C302 pad 2: Net-(C301-Pad2) -> Net-(C302-Pad2)
- C303 pad 1: Net-(C301-Pad2) -> /Mic Path/Mic2
- C303 pad 2: Net-(C303-Pad2) -> Net-(C302-Pad2)
- C304 pad 1: Net-(C302-Pad1) -> Net-(C302-Pad2)
- C304 pad 2: Net-(C304-Pad2) -> /Mic Path/Mic3
- C305 pad 1: Net-(C303-Pad2) -> /Mic Path/Mic2
- C306 pad 1: Net-(C306-Pad1) -> /Mic Path/Mic3
- C306 pad 2: Net-(D303-A) -> Net-(C306-Pad2)
- C307 pad 1: +5V -> Net-(C307-Pad1)
- C307 pad 2: GND -> /Mic Path/RG2
- C308 pad 1: -5V -> GND
- C308 pad 2: GND -> +5V
- C309 pad 1: -5V -> GND
- C309 pad 2: +5V -> -5V
- C310 pad 1: GND -> +5V
- C310 pad 2: +5V -> GND
- C311 pad 1: GND -> -5V
- C311 pad 2: -5V -> GND
- C312 pad 2: +5V -> Net-(C312-Pad2)
- C313 pad 2: -5V -> Net-(C313-Pad2)
- C314 pad 2: Net-(C314-Pad2) -> +5V
- C315 pad 2: Net-(C315-Pad2) -> -5V
- C316 pad 2: Net-(U304-OUT+) -> /Mic Path/MicOut+
- C317 pad 2: Net-(U304-OUT-) -> /Mic Path/MicOut-
- C318 pad 1: Net-(C318-Pad1) -> /Mic Path/MicOut2
- C319 pad 2: Net-(C319-Pad2) -> /Mic Path/MicOut3
- C405 pad 1: Net-(J403-Pin_2) -> Net-(J405-Pin_2)
- C406 pad 1: Net-(J404-Pin_2) -> Net-(J403-Pin_2)
- C407 pad 1: GND -> Net-(U403A-+)
- C407 pad 2: Net-(D406-A) -> Net-(C407-Pad2)
- C408 pad 1: Net-(U403A-+) -> Net-(U403B-+)
- C409 pad 1: Net-(U403B-+) -> GND
- C409 pad 2: Net-(C409-Pad2) -> Net-(D405-A)
- D301 pad 2: Net-(D302-K) -> /Mic Path/Micpre+
- D301 pad 3: Net-(D303-K) -> /Mic Path/Micpre-
- D302 pad 1: Net-(D302-K) -> +5V
- D302 pad 2: Net-(D302-A) -> GND
- D303 pad 1: Net-(D303-K) -> GND
- D303 pad 2: Net-(D303-A) -> -5V
- D304 pad 1: +5V -> /Mic Path/Micpre+
- D304 pad 2: GND -> /Mic Path/RG1
- D305 pad 1: GND -> /Mic Path/Micpre-
- D305 pad 2: -5V -> /Mic Path/RG2
- D306 pad 1: -5V -> Net-(D306-K)
- D306 pad 2: Net-(D306-Pad2) -> Net-(D306-A)
- D307 pad 2: Net-(U304-OUT+) -> /Mic Path/MicOut+
- D307 pad 3: Net-(U304-OUT-) -> /Mic Path/MicOut-
- D308 pad 1: Net-(D308-K) -> -5V
- D308 pad 2: Net-(D308-A) -> Net-(D308-Pad2)
- FB301 pad 1: Net-(D306-Pad2) -> /Mic Path/MicOut+
- FB301 pad 2: Net-(C318-Pad1) -> /Mic Path/MicOut2
- FB302 pad 1: Net-(D306-Pad3) -> /Mic Path/MicOut-
- FB302 pad 2: Net-(C319-Pad2) -> /Mic Path/MicOut3
- FB303 pad 1: Net-(U304-OUT+) -> Net-(D308-Pad2)
- FB304 pad 1: Net-(U304-OUT-) -> Net-(D308-Pad3)
- J301 pad 2: Net-(C302-Pad1) -> /Mic Path/Mic2
- J301 pad 3: Net-(C303-Pad2) -> /Mic Path/Mic3
- J302 pad 2: Net-(D308-K) -> Net-(J302-Pin_2)
- J303 pad 2: Net-(J303-Pin_2) -> Net-(D306-A)
- J304 pad 2: Net-(D308-A) -> Net-(D306-K)
- J306 pad 2: Net-(C318-Pad1) -> Net-(C320-Pad1)
- J306 pad 3: Net-(C319-Pad2) -> Net-(C321-Pad2)
- J307 pad 2: Net-(C320-Pad1) -> /Mic Path/MicOut2
- J307 pad 3: Net-(C321-Pad2) -> /Mic Path/MicOut3
- J404 pad 3: GND -> Net-(J404-Pin_3-Pad3)
- J405 pad 3: Net-(J405-Pin_3) -> GND
- J406 pad R: Net-(C409-Pad2) -> Net-(C408-Pad2)
- J406 pad T: Net-(C408-Pad2) -> Net-(C407-Pad2)
- J407 pad T: Net-(C408-Pad2) -> Net-(C407-Pad2)
- R205 pad 1: Net-(Q201-B) -> Net-(U201-FB)
- R205 pad 2: Net-(D202-A) -> GND
- R206 pad 1: Net-(U201-FB) -> Net-(U202-FB)
- R206 pad 2: GND -> -5V
- R207 pad 1: Net-(U202-FB) -> Net-(U201-FB)
- R207 pad 2: -5V -> +5V
- R208 pad 1: Net-(U201-FB) -> Net-(U202-FB)
- R208 pad 2: +5V -> GND
- R301 pad 1: Net-(D302-K) -> /Mic Path/Micpre+
- R301 pad 2: Net-(C304-Pad2) -> Net-(C305-Pad2)
- R302 pad 1: Net-(D303-K) -> /Mic Path/Micpre-
- R302 pad 2: Net-(C305-Pad2) -> Net-(C306-Pad2)
- R303 pad 1: Net-(D302-K) -> /Mic Path/Micpre+
- R304 pad 2: Net-(D303-K) -> /Mic Path/Micpre-
- R306 pad 1: Net-(C306-Pad1) -> Net-(C307-Pad1)
- R306 pad 2: Net-(D302-A) -> /Mic Path/RG1
- R307 pad 1: Net-(J302-Pin_1) -> Net-(J303-Pin_1)
- R309 pad 1: Net-(U302B-D) -> Net-(D306-K)
- R309 pad 2: Net-(U303A-+) -> -5V
- R310 pad 1: Net-(D306-Pad2) -> Net-(D306-A)
- R310 pad 2: Net-(U303A-+) -> -5V
- R311 pad 1: Net-(R311-Pad1) -> Net-(U301B-D)
- R311 pad 2: Net-(D306-Pad2) -> Net-(U302A-+)
- R312 pad 1: Net-(R311-Pad1) -> Net-(U301B-D)
- R312 pad 2: Net-(U303A--) -> Net-(U302B--)
- R313 pad 1: Net-(C314-Pad2) -> Net-(C312-Pad2)
- R313 pad 2: Net-(U303A--) -> Net-(U302A--)
- R314 pad 1: Net-(U302B-D) -> Net-(C313-Pad2)
- R314 pad 2: Net-(U303B--) -> Net-(U302B-+)
- R315 pad 1: Net-(C315-Pad2) -> Net-(D308-Pad2)
- R315 pad 2: Net-(U303B-+) -> Net-(U302A-+)
- R316 pad 2: Net-(U303B--) -> Net-(U302A--)
- R317 pad 1: Net-(D306-Pad3) -> Net-(R317-Pad1)
- R317 pad 2: Net-(U303B-+) -> Net-(U302B--)
- R318 pad 1: Net-(R316-Pad1) -> Net-(D308-Pad3)
- R318 pad 2: Net-(D306-Pad3) -> Net-(U302B-+)
- R319 pad 1: Net-(D308-A) -> Net-(R316-Pad1)
- R319 pad 2: -5V -> Net-(D308-Pad2)
- R320 pad 1: Net-(D308-K) -> Net-(R317-Pad1)
- R320 pad 2: -5V -> Net-(D308-Pad3)
- R405 pad 1: +5V -> Net-(J405-Pin_2)
- R405 pad 2: Net-(J403-Pin_1) -> Net-(R405-Pad2)
- R406 pad 1: +5V -> Net-(R405-Pad2)
- R406 pad 2: Net-(J404-Pin_1) -> Net-(J403-Pin_2)
- R407 pad 2: Net-(R407-Pad2) -> Net-(J403-Pin_1)
- R408 pad 1: Net-(U403A-+) -> +5V
- R408 pad 2: Net-(C408-Pad2) -> Net-(J405-Pin_1)
- R409 pad 1: Net-(U403B-+) -> +5V
- R409 pad 2: Net-(C409-Pad2) -> Net-(R405-Pad2)
- R410 pad 1: Net-(D406-A) -> GND
- R410 pad 2: +5V -> Net-(R405-Pad2)
- R411 pad 1: GND -> Net-(U403A-+)
- R411 pad 2: Net-(R407-Pad2) -> Net-(C407-Pad2)
- R412 pad 1: Net-(J403-Pin_2) -> Net-(U403B-+)
- R412 pad 2: Net-(R407-Pad2) -> Net-(C408-Pad2)
- R413 pad 1: Net-(R407-Pad2) -> Net-(D405-A)
- R413 pad 2: Net-(J404-Pin_2) -> +5V
- RV402 pad 1: Net-(J405-Pin_1) -> Net-(J404-Pin_1)
- RV402 pad 2: Net-(J405-Pin_2) -> Net-(J404-Pin_2)
- RV402 pad 3: Net-(J405-Pin_3) -> Net-(J404-Pin_3-Pad3)
- SW301 pad 1: Net-(J303-Pin_1) -> Net-(J302-Pin_1)
- SW301 pad 2: Net-(J303-Pin_2) -> Net-(J302-Pin_2)
- U301 pad 1: Net-(D302-A) -> Net-(D306-K)
- U301 pad 2: Net-(D303-K) -> GND
- U301 pad 3: Net-(D302-K) -> /Mic Path/MicOut
- U301 pad 4: -5V -> /Mic Path/MicpreOut
- U301 pad 5: GND -> +5V
- U301 pad 6: Net-(U301-Out) -> GND
- U301 pad 7: +5V -> unconnected-(U301C-NC-Pad7)
- U301 pad 8: Net-(D303-A) -> unconnected-(U301C-NC-Pad8)
- U302 pad 1: Net-(D308-K) -> Net-(R316-Pad1)
- U302 pad 2: GND -> Net-(U302A--)
- U302 pad 3: Net-(U302A-D) -> Net-(U302A-+)
- U302 pad 4: Net-(U301-Out) -> -5V
- U302 pad 5: +5V -> Net-(U302B-+)
- U302 pad 6: GND -> Net-(U302B--)
- U302 pad 7: unconnected-(U302C-NC-Pad7) -> Net-(R317-Pad1)
- U302 pad 8: unconnected-(U302C-NC-Pad8) -> +5V
- U302 pad 9: Net-(D308-A) -> -5V
- U303 pad 1: Net-(R311-Pad1) -> /Mic Path/RG1
- U303 pad 2: Net-(U303A--) -> /Mic Path/Micpre-
- U303 pad 3: Net-(U303A-+) -> /Mic Path/Micpre+
- U303 pad 5: Net-(U303B-+) -> GND
- U303 pad 6: Net-(U303B--) -> /Mic Path/MicpreOut
- U303 pad 7: Net-(R316-Pad1) -> +5V
- U303 pad 8: +5V -> /Mic Path/RG2
- U304 pad 1: Net-(U304-OUT-) -> /Mic Path/MicOut-
- U304 pad 4: Net-(U302A-D) -> /Mic Path/MicOut
- U304 pad 8: Net-(U304-OUT+) -> /Mic Path/MicOut+
- U402 pad 3: Net-(J403-Pin_2) -> Net-(J405-Pin_2)
- U402 pad 5: Net-(J404-Pin_2) -> Net-(J403-Pin_2)
- U403 pad 7: Net-(C409-Pad2) -> Net-(C408-Pad2)
- U403 pad 8: Net-(D406-A) -> Net-(D405-A)
- U403 pad 9: Net-(C408-Pad2) -> Net-(C407-Pad2)
Other:
- board outline added: 106 x 93 mm

Commit message: progress
Parts:
- added C209: 100n, Capacitor_SMD:C_0402_1005Metric, F.Cu at (169.5, 101.7)
- added C322: 100n, Capacitor_SMD:C_0402_1005Metric, F.Cu at (116.6, 82.0)
- R312: value 10k -> 20k
- SW301, SW302: moved to B.Cu
- moved R410 46.8 mm to (154.5, 100.0), turned to -90 degrees
- moved C406 45.6 mm to (152.4, 102.4), turned to 90 degrees
- moved R409 44.6 mm to (155.5, 100.0), turned to -90 degrees
- moved C412 42.7 mm to (155.0, 105.8)
- moved C413 41.7 mm to (155.0, 101.4)
- moved C405 41.2 mm to (157.6, 102.9), turned to 90 degrees
- moved R405 41.0 mm to (158.5, 102.9), turned to 90 degrees
- moved R406 40.4 mm to (151.5, 102.4), turned to -90 degrees
- moved J305 37.8 mm to (232.0, 96.2)
- moved U402 37.5 mm to (155.0, 103.6), turned to 180 degrees
- moved D201 32.6 mm to (175.5, 82.6), turned to -90 degrees
- moved R207 31.8 mm to (165.5, 110.0), turned to 90 degrees
- moved U403 30.4 mm to (155.0, 114.8), turned to -90 degrees
- moved D203 28.4 mm to (181.5, 82.2), turned to 90 degrees
- moved C415 27.9 mm to (156.1, 112.2)
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Connections:
- net Net-(D202-K) renamed /Power/vbulk
- net Net-(D306-A) renamed /Mic Path/TBSel
- net Net-(D306-K) renamed /Mic Path/MuteSel
- net Net-(U301B-D) renamed /Mic Path/TBOut
- C301 pad 2: +5V -> GND
- C407 pad 1: Net-(U403A-+) -> Net-(U401A-OUT)
- C408 pad 1: Net-(U403B-+) -> Net-(U401B-OUT)
- D301 pad 2: /Mic Path/Micpre+ -> /Mic Path/Micpre-
- D301 pad 3: /Mic Path/Micpre- -> /Mic Path/Micpre+
- D307 pad 2: /Mic Path/MicOut+ -> /Mic Path/MicOut-
- D307 pad 3: /Mic Path/MicOut- -> /Mic Path/MicOut+
- R411 pad 1: Net-(U403A-+) -> Net-(U401A-OUT)
- R412 pad 1: Net-(U403B-+) -> Net-(U401B-OUT)
- U301 pad 13: -5V -> +5V
- U301 pad 5: +5V -> -5V
- U403 pad 1: Net-(U403A-+) -> GND
- U403 pad 5: Net-(U403B-+) -> GND
Routing:
- net /Power/vbulk: track 0.00 -> 51.8 mm
- net /Mic Path/Micpre-: track 0.00 -> 30.3 mm
- net IFB_PIN2: track 0.00 -> 24.5 mm
- net Net-(C407-Pad2): track 0.00 -> 21.6 mm
- net +5V: track 0.00 -> 20.6 mm, vias 0 -> 1
- net GND: track 0.00 -> 20.3 mm, vias 0 -> 31
- net /Mic Path/Micpre+: track 0.00 -> 18.4 mm
- net -5V: track 0.00 -> 18.3 mm, vias 0 -> 1
- net /Mic Path/Mic2: track 0.00 -> 13.4 mm
- net /Mic Path/MicOut+: track 0.00 -> 12.8 mm
- net /Mic Path/MicOut-: track 0.00 -> 11.7 mm
- net Net-(U401B-OUT): track 0.00 -> 10.4 mm
- net Net-(U401A-OUT): track 0.00 -> 10.1 mm
- net Net-(R405-Pad2): track 0.00 -> 9.62 mm
- net /Mic Path/Mic3: track 0.00 -> 8.90 mm
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- added copper zone on F.Cu, net GND
- added copper zone on In1.Cu, net GND
- added copper zone on F.Cu, net Net-(U201-SW)
- added copper zone on F.Cu, net Net-(U202-SW)
Other:
- copper layers 2 -> 4

Commit message: Moar Progress
Parts:
- added H105: Mousebites, STEVEannouncer:Mousebites, F.Cu at (167.0, 136.0)
- added H106: Mousebites, STEVEannouncer:Mousebites, F.Cu at (167.0, 134.0)
- added H107: Mousebites, STEVEannouncer:Mousebites, F.Cu at (187.0, 134.0)
- added H108: Mousebites, STEVEannouncer:Mousebites, F.Cu at (187.0, 136.0)
- added H109: Mousebites, STEVEannouncer:Mousebites, F.Cu at (160.0, 144.0)
- added H110: Mousebites, STEVEannouncer:Mousebites, F.Cu at (174.0, 144.0)
- added H111: Mousebites, STEVEannouncer:Mousebites, F.Cu at (180.0, 144.0)
- added H112: Mousebites, STEVEannouncer:Mousebites, F.Cu at (154.0, 144.0)
- added H113: Mousebites, STEVEannouncer:Mousebites, F.Cu at (160.0, 123.0)
- added H114: Mousebites, STEVEannouncer:Mousebites, F.Cu at (154.0, 123.0)
- added H115: Mousebites, STEVEannouncer:Mousebites, F.Cu at (167.0, 116.0)
- added H116: Mousebites, STEVEannouncer:Mousebites, F.Cu at (187.0, 116.0)
- added H117: Mousebites, STEVEannouncer:Mousebites, F.Cu at (167.0, 114.0)
- added H118: Mousebites, STEVEannouncer:Mousebites, F.Cu at (187.0, 114.0)
- added H119: Mousebites, STEVEannouncer:Mousebites, F.Cu at (179.8, 123.0)
- added H120: Mousebites, STEVEannouncer:Mousebites, F.Cu at (174.0, 123.0)
- J301, J401: footprint Connector_Audio:Jack_XLR_Neutrik_NC3FAH2_Horizontal -> STEVEannouncer:NC3FAH2
- J302, J305: moved to B.Cu
- J306, J307: footprint Connector_Audio:Jack_XLR_Neutrik_NC3MAH_Horizontal -> STEVEannouncer:NC3MAH
- J406, J407: footprint Connector_Audio:Jack_6.35mm_Neutrik_NRJ6HF_Horizontal -> STEVEannouncer:NRJ6HF
- SW301, SW302: footprint Button_Switch_Keyboard:SW_Cherry_MX_1.00u_PCB -> STEVEannouncer:CherrySwitch; moved to F.Cu
- moved J404 148.9 mm to (187.0, 141.0)
- moved J403 139.7 mm to (25.4, 110.8)
- moved J405 138.3 mm to (25.4, 129.8)
- moved RV402 132.6 mm to (187.0, 148.2)
- moved J402 132.0 mm to (167.0, 141.0)
- moved RV401 118.4 mm to (167.0, 148.2)
- moved J302 91.4 mm to (167.0, 130.0), turned to 180 degrees
- moved SW301 65.9 mm to (169.5, 117.9)
- moved J305 56.2 mm to (187.0, 130.0), turned to 180 degrees
- moved H103 55.5 mm to (135.0, 123.0)
- moved SW302 46.3 mm to (189.5, 117.9)
- moved H102 27.9 mm to (118.0, 82.0)
- moved D306 19.3 mm to (130.0, 118.1)
- moved R309 19.3 mm to (130.0, 116.0)
- moved R310 19.3 mm to (130.0, 120.0)
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Routing:
- net /Mic Path/MicpreOut: track 0.00 -> 38.9 mm
- net /Mic Path/MuteSel: track 0.00 -> 28.9 mm, vias 0 -> 2
- net /Mic Path/TBSel: track 0.00 -> 22.2 mm
- net /Mic Path/TBOut: track 0.00 -> 20.1 mm
- net /Power/vbulk: track 51.8 -> 37.0 mm
- net Net-(J305-Pin_1): track 0.00 -> 13.2 mm
- net Net-(J302-Pin_1): track 0.00 -> 13.2 mm
- net Net-(J305-Pin_2): track 0.00 -> 11.2 mm
- net Net-(J302-Pin_2): track 0.00 -> 11.2 mm
- net Net-(J404-Pin_3-Pad3): track 0.00 -> 7.94 mm
- net Net-(J404-Pin_1): track 0.00 -> 7.94 mm
- net Net-(J402-Pin_3-Pad3): track 0.00 -> 7.94 mm
- net Net-(J402-Pin_1): track 0.00 -> 7.94 mm
- net GND: track 20.3 -> 28.2 mm, vias 31 -> 35
- net /Mic Path/MicOut: track 0.00 -> 7.35 mm
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Other:
- board size 106 x 93 mm -> 110 x 86 mm
- board text added: "Mute"
- board text added: "Talkback"

Commit message: Even more more progress
Parts:
- added C323: 100n, Capacitor_SMD:C_0402_1005Metric, F.Cu at (123.0, 99.5)
- added C324: 100n, Capacitor_SMD:C_0402_1005Metric, F.Cu at (113.5, 99.5)
- added C416: 100p, Capacitor_SMD:C_0402_1005Metric, F.Cu at (172.0, 86.8)
- added C417: 100p, Capacitor_SMD:C_0402_1005Metric, F.Cu at (170.0, 86.8)
- added FB401: FerriteBead, Inductor_SMD:L_0402_1005Metric, F.Cu at (173.5, 87.2)
- added FB402: FerriteBead, Inductor_SMD:L_0402_1005Metric, F.Cu at (168.5, 87.2)
- added FID101: Fiducial, Fiducial:Fiducial_1mm_Mask3mm, F.Cu at (91.0, 142.0)
- added FID102: Fiducial, Fiducial:Fiducial_1mm_Mask3mm, F.Cu at (91.0, 77.0)
- added FID103: Fiducial, Fiducial:Fiducial_1mm_Mask3mm, F.Cu at (193.0, 77.0)
- moved J403 129.3 mm to (153.2, 91.1)
- moved J405 122.3 mm to (141.4, 91.1)
- moved H103 59.4 mm to (193.0, 110.0)
- moved D302 44.2 mm to (94.5, 99.5)
- moved D303 44.2 mm to (94.5, 102.0)
- moved R408 31.5 mm to (137.8, 96.2), turned to 90 degrees
- moved H102 29.5 mm to (91.0, 70.0)
- moved R407 27.1 mm to (149.7, 96.2), turned to 90 degrees
- moved R309 22.6 mm to (113.5, 100.5)
- moved D306 21.6 mm to (117.5, 100.5)
- moved R310 20.7 mm to (123.0, 100.5)
- moved H101 14.8 mm to (91.0, 148.0)
- moved C402 13.8 mm to (134.8, 107.0), turned to -90 degrees
- moved R401 11.3 mm to (143.2, 108.9), turned to -90 degrees
- moved R406 11.3 mm to (135.8, 101.4)
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Connections:
- net Net-(C320-Pad1) renamed /Mic Path/TB_OUT2
- net Net-(C321-Pad2) renamed /Mic Path/TB_OUT3
- net Net-(C407-Pad2) renamed /IFB Path/HP_L
- net Net-(C408-Pad2) renamed /IFB Path/HP_R
- net Net-(D401-A) renamed /IFB Path/VCA_INL
- net Net-(D402-A) renamed /IFB Path/VCA_INR
- net Net-(U401A-E-) renamed /IFB Path/VCAL_E-
- net Net-(U401A-OUT) renamed /IFB Path/VCA_OUTL
- net Net-(U401B-E-) renamed /IFB Path/VCAR_E-
- net Net-(U401B-OUT) renamed /IFB Path/VCA_OUTR
- C402 pad 1: Net-(C402-Pad1) -> /IFB Path/IFB_Pin3
- J401 pad 2: IFB_PIN2 -> Net-(C416-Pad1)
- J401 pad 3: Net-(C402-Pad1) -> Net-(C417-Pad2)
Routing:
- net /IFB Path/IFB_Pin3: track 0.00 -> 41.5 mm
- net IFB_PIN2: track 17.3 -> 50.3 mm
- net Net-(J403-Pin_2): track 0.00 -> 30.6 mm
- net /IFB Path/HP_R: track 1.87 -> 31.8 mm
- net /Power/vbulk: track 37.0 -> 62.5 mm
- net /IFB Path/HP_L: track 21.6 -> 40.8 mm
- net Net-(J405-Pin_2): track 1.20 -> 14.7 mm
- net Net-(C416-Pad1): track 0.00 -> 8.74 mm
- net /IFB Path/VCA_INL: track 0.00 -> 6.55 mm
- net /Mic Path/TBSel: track 22.2 -> 16.8 mm
- net /IFB Path/VCA_INR: track 0.00 -> 5.14 mm
- net Net-(C417-Pad2): track 0.00 -> 4.87 mm
- net Net-(J405-Pin_1): track 0.00 -> 4.68 mm
- net Net-(J403-Pin_1): track 0.00 -> 4.66 mm
- net Net-(D405-A): track 2.97 -> 6.88 mm
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- added copper zone on F.Cu, net +5V
- added copper zone on F.Cu, net -5V
Other:
- board text added: "+"
- board text added: "10k Linear Pots"
- board text added: "12-24 VDC"
- board text added: "CCW"
- board text added: "CW"
- board text added: "Full schematics and other repair info at https://github.com/Solomute/STEVEannouncer"
- board text added: "Int (L)"
- board text added: "Mechanical Keyboard Switches (i.e. Cherry MX)"
- board text added: "Mute (L)"
- board text added: "Non-Int (R)"
- board text added: "Talkback (R)"
- board text added: "Wiper"
- board text removed: "Mute"
- board text removed: "Talkback"

Commit message: Yeet
Parts:
- added D204: LED, LED_SMD:LED_0603_1608Metric, F.Cu at (149.8, 67.0)
- added R209: 1k, Resistor_SMD:R_0402_1005Metric, F.Cu at (151.0, 69.0)
- H101, H102, H103, H104: footprint MountingHole:MountingHole_3.2mm_M3 -> MountingHole:MountingHole_3.2mm_M3_Pad_TopBottom
- J401: value ~ -> NC3FAH2
- moved D303 4.78 mm to (99.3, 102.0), turned to 180 degrees
- moved D302 4.77 mm to (99.3, 99.4)
Routing:
- net GND: track 29.6 -> 54.1 mm, vias 38 -> 66
- net +5V: track 20.6 -> 39.7 mm, vias 3 -> 22
- net /IFB Path/VCAR_E-: track 0.50 -> 12.1 mm, vias 0 -> 2
- net -5V: track 19.4 -> 30.5 mm, vias 3 -> 16
- net /IFB Path/VCAL_E-: track 0.50 -> 10.9 mm, vias 0 -> 2
- net Net-(D308-Pad3): track 5.00 -> 13.0 mm, vias 0 -> 2
- net Net-(D204-A): track 0.00 -> 1.67 mm
- net /Mic Path/MicpreOut: track 38.4 -> 38.9 mm
- added copper zone on B.Cu, net +5V
- added copper zone on B.Cu, net -5V
- added copper zone on In2.Cu, net GND
Other:
- board text added: "IFB In"
- board text added: "Mic In"
- board text added: "Mic Out"
- board text added: "Mono Headphone"
- board text added: "Stereo Headphone"
- board text added: "TB Out"
