File: PCB/STEVEannouncer.kicad_pcb (KiCad board)
At the start: 4 copper layers, 110 x 86 mm, 170 parts, among them J201 Barrel_Jack_Switch, J301 NC3FAH, J302 Conn_01x02, J303 Conn_01x02, J304 Conn_01x02, J305 Conn_01x02, J306 NC3MAH, J307 NC3MAH, J401 NC3FAH2, J402 Conn_01x03, J403 Conn_01x03, J404 Conn_01x03, J405 Conn_01x03, J406 NRJ6HF, J407 NRJ6HF, Q201 BC847, Q202 BCV49, SW301 SW_SPST, SW302 SW_SPST, U201 LV3842, U202 LV3842, U301 TMUX6236, U302 OPA1678, U303 THAT1512, U304 THAT1646, U401 THAT2162, U402 OPA1678, U403 OPA1622

Commit message: I think I can fab this????
Parts:
- J302, J305: moved to F.Cu
- SW301, SW302: moved to B.Cu
- U201, U202: footprint Package_TO_SOT_SMD:SOT-23-6 -> STEVEannouncer:SOT-23-6
- U302, U402: footprint Package_SON:WSON-8-1EP_3x3mm_P0.5mm_EP1.2x2mm_ThermalVias -> STEVEannouncer:WSON-8-1EP_3x3mm_P0.5mm_EP1.2x2mm_ThermalVias
- U403: footprint Package_SON:Texas_S-PVSON-N10_ThermalVias -> STEVEannouncer:OPA1622
- moved SW301 5.08 mm to (164.5, 117.9), turned to 180 degrees
- moved SW302 5.08 mm to (184.5, 117.9), turned to 180 degrees
- moved J406 0.05 mm to (134.4, 135.1)
- moved J407 0.05 mm to (151.4, 135.1)
- turned J302 to 0 degrees
- turned J305 to 0 degrees
Connections:
- R309 pad 2: -5V -> GND
- R310 pad 2: -5V -> GND
Routing:
- net +5V: track 39.7 -> 33.5 mm, vias 22 -> 25
- net Net-(J405-Pin_1): track 4.68 -> 2.19 mm
- net GND: track 54.1 -> 56.6 mm, vias 66 -> 68
- net /Power/vbulk: track 62.5 -> 60.5 mm
- net -5V: track 30.5 -> 29.1 mm, vias 16 -> 17
- net Net-(C416-Pad1): track 8.74 -> 7.74 mm
- net /IFB Path/HP_L: track 40.8 -> 39.8 mm
- net Net-(D203-A): track 6.53 -> 5.61 mm
- net /Mic Path/MicOut2: track 4.00 -> 3.23 mm
- net /Mic Path/MicOut3: track 4.01 -> 3.26 mm
- net Net-(C417-Pad2): track 4.87 -> 4.14 mm
- net /Mic Path/Micpre+: track 18.4 -> 17.7 mm
- net Net-(J305-Pin_1): track 13.6 -> 12.9 mm
- net Net-(J302-Pin_1): track 13.6 -> 12.9 mm
- net /Mic Path/MicOut-: track 11.7 -> 11.1 mm
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- added copper zone on F.Cu, net /Power/vbulk
Other:
- board text added: "Designed by Stephan Ahonen Revision 2025-06-30 Full schematics and other repair info at https://github.com/Solomute/STEVEannouncer"
- board text removed: "Full schematics and other repair info at https://github.com/Solomute/STEVEannouncer"

Commit message: There, I ordered it
Parts:
- D306: value BAS716 -> D_Schottky
- J301: value NC3FAH -> NC3FAH2
- R307, R308: value 330k -> 20k
- SW301, SW302: footprint STEVEannouncer:CherrySwitch -> STEVEannouncer:SW_choc_v1_1u
- moved SW301 5.68 mm to (167.0, 123.0), turned to 0 degrees
- moved SW302 5.68 mm to (187.0, 123.0), turned to 0 degrees
- moved J302 1.25 mm to (166.0, 129.2), turned to 180 degrees
- moved J305 1.25 mm to (186.0, 129.2), turned to 180 degrees
- moved H115 0.25 mm to (167.0, 115.8)
- moved H116 0.25 mm to (187.0, 115.8)
- moved H119 0.20 mm to (180.0, 123.0)
- turned D306 to 180 degrees
Connections:
- D306 pad 1: /Mic Path/MuteSel -> /Mic Path/TBSel
- D306 pad 2: /Mic Path/TBSel -> /Mic Path/MuteSel
- R307 pad 2: +5V -> GND
- R308 pad 2: +5V -> GND
- R309 pad 2: GND -> +5V
- R310 pad 2: GND -> +5V
- SW301 pad 1: Net-(J302-Pin_1) -> Net-(J302-Pin_2)
- SW301 pad 2: Net-(J302-Pin_2) -> Net-(J302-Pin_1)
- SW302 pad 1: Net-(J305-Pin_1) -> Net-(J305-Pin_2)
- SW302 pad 2: Net-(J305-Pin_2) -> Net-(J305-Pin_1)
- U301 pad 10: /Mic Path/MicpreOut -> GND
- U301 pad 12: GND -> /Mic Path/MicpreOut
- U301 pad 2: GND -> /Mic Path/MicpreOut
- U301 pad 4: /Mic Path/MicpreOut -> GND
Routing:
- net Net-(J302-Pin_1): track 12.9 -> 15.0 mm
- net GND: track 56.6 -> 58.5 mm
- net Net-(J305-Pin_1): track 12.9 -> 14.8 mm
- net /Mic Path/MicpreOut: track 38.9 -> 40.1 mm
Other:
- outline, holes or cut-outs redrawn
- board text added: "Designed by Stephan Ahonen Revision 2025-07-01 Full schematics and other repair info at https://github.com/Solomute/STEVEannouncer"
- board text removed: "Designed by Stephan Ahonen Revision 2025-06-30 Full schematics and other repair info at https://github.com/Solomute/STEVEannouncer"
