File: PCB/STEVEannouncer.kicad_pcb (KiCad board)
At the start: 4 copper layers, 110 x 86 mm, 170 parts, among them J201 Barrel_Jack_Switch, J301 NC3FAH2, J302 Conn_01x02, J303 Conn_01x02, J304 Conn_01x02, J305 Conn_01x02, J306 NC3MAH, J307 NC3MAH, J401 NC3FAH2, J402 Conn_01x03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

Commit message: revisionnnnn
Parts:
- added C325: 100n, Capacitor_SMD:C_0402_1005Metric, F.Cu at (72.6, 125.1)
- added C326: 100n, Capacitor_SMD:C_0402_1005Metric, F.Cu at (72.6, 127.1)
- added C327: 10u, Capacitor_SMD:C_0603_1608Metric, F.Cu at (69.2, 125.4)
- added R210: 80.6k, Resistor_SMD:R_0402_1005Metric, F.Cu at (78.7, 120.5)
- added R211: 10k, Resistor_SMD:R_0402_1005Metric, F.Cu at (78.7, 122.5)
- added R321: 10k, Resistor_SMD:R_0402_1005Metric, F.Cu at (73.8, 120.5)
- added R322: 10k, Resistor_SMD:R_0402_1005Metric, F.Cu at (73.8, 122.5)
- added U305: OPA202, Package_TO_SOT_SMD:SOT-23-5, F.Cu at (111.3, 117.7)
Connections:
- C313 pad 1: GND -> Net-(C313-Pad1)
- C313 pad 2: Net-(C313-Pad2) -> /Mic Path/TBOut
- R312 pad 1: /Mic Path/TBOut -> Net-(C313-Pad1)
- R314 pad 1: Net-(C313-Pad2) -> GND
- U201 pad 4: /Power/vbulk -> Net-(U201-EN)
- U202 pad 4: /Power/vbulk -> +5V
- U303 pad 5: GND -> Net-(U303-Ref)
Routing:
- net GND: track 58.5 -> 56.4 mm, vias 68 -> 66
- net Net-(C313-Pad2): track 0.86 -> 0.00 mm
- net (no net): track 0.00 -> 0.86 mm
- net Net-(C313-Pad1): track 0.00 -> 0.72 mm, vias 0 -> 1

Commit message: Rev 2025-07-20
Parts:
- added C328: 470p, Capacitor_SMD:C_0402_1005Metric, F.Cu at (111.0, 92.0)
- added C329: 470p, Capacitor_SMD:C_0402_1005Metric, F.Cu at (122.1, 93.2)
- D301, D307, D308: value BAS3007ARPPE6327HTSA1 -> BAS3007
- J302, J305: footprint Connector_JST:JST_PH_B2B-PH-SM4-TB_1x02-1MP_P2.00mm_Vertical -> STEVEannouncer:SolderWire-0.15sqmm_1x02_P4mm_D0.5mm_OD1.5mm
- J402, J404: footprint Connector_JST:JST_PH_B3B-PH-SM4-TB_1x03-1MP_P2.00mm_Vertical -> Connector_Wire:SolderWire-0.15sqmm_1x03_P4mm_D0.5mm_OD1.5mm
- Q202: footprint Package_TO_SOT_SMD:SOT-89-3 -> STEVEannouncer:SOT-89-3
- R306: value 270 -> 100
- moved R211 93.1 mm to (171.2, 112.2), turned to 90 degrees
- moved R210 93.1 mm to (171.2, 110.3), turned to 90 degrees
- moved C327 44.2 mm to (112.4, 116.2), turned to -90 degrees
- moved C326 38.9 mm to (109.0, 113.2), turned to -90 degrees
- moved R321 37.8 mm to (110.8, 113.2), turned to -90 degrees
- moved C325 37.7 mm to (109.9, 119.2), turned to 90 degrees
- moved R322 37.2 mm to (110.8, 119.2), turned to -90 degrees
- moved J305 8.55 mm to (188.5, 121.1)
- moved J302 8.52 mm to (168.5, 121.1)
- moved D201 7.70 mm to (169.2, 92.5)
- moved R203 4.40 mm to (170.5, 95.6), turned to 0 degrees
- moved J402 4.12 mm to (163.0, 140.0)
- moved J404 4.12 mm to (183.0, 140.0)
- moved H105 4.03 mm to (170.5, 138.0)
- moved H108 4.03 mm to (190.5, 138.0)
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Connections:
- net Net-(D202-A) renamed /Power/Pin2_Bulk
- C201 pad 1: Net-(Q201-C) -> /Power/Darl_B
- Q201 pad 1: Net-(Q201-B) -> /Power/Darl_E
- Q201 pad 3: Net-(Q201-C) -> /Power/Darl_B
- Q202 pad 1: Net-(Q201-B) -> /Power/Darl_B
- Q202 pad 3: Net-(Q201-C) -> /Power/Darl_E
- R201 pad 2: Net-(Q201-C) -> /Power/Darl_B
- R202 pad 1: Net-(Q201-C) -> /Power/Darl_B
- R203 pad 2: Net-(Q201-C) -> /Power/Darl_B
- R204 pad 1: Net-(Q201-B) -> /Power/Darl_E
- SW301 pad 1: Net-(J302-Pin_2) -> Net-(J302-Pin_1)
- SW301 pad 2: Net-(J302-Pin_1) -> Net-(J302-Pin_2)
- SW302 pad 1: Net-(J305-Pin_2) -> Net-(J305-Pin_1)
- SW302 pad 2: Net-(J305-Pin_1) -> Net-(J305-Pin_2)
Routing:
- net +5V: track 33.5 -> 55.2 mm, vias 25 -> 27
- net GND: track 56.4 -> 67.1 mm, vias 66 -> 70
- net Net-(U303-Ref): track 0.00 -> 10.2 mm
- net /Power/Darl_B: track 0.00 -> 10.0 mm
- net -5V: track 29.1 -> 35.7 mm, vias 17 -> 18
- net Net-(Q201-C): track 6.42 -> 0.00 mm
- net Net-(J302-Pin_1): track 15.0 -> 10.1 mm
- net Net-(Q201-B): track 4.60 -> 0.00 mm
- net Net-(J305-Pin_1): track 14.8 -> 10.2 mm
- net /Mic Path/MicpreOut: track 40.1 -> 44.3 mm
- net Net-(U305--): track 0.00 -> 4.10 mm
- net /Power/Darl_E: track 0.00 -> 3.89 mm
- net Net-(U201-EN): track 0.00 -> 3.71 mm
- net Net-(J305-Pin_2): track 10.8 -> 13.5 mm
- net Net-(J302-Pin_2): track 10.8 -> 13.5 mm
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Other:
- outline, holes or cut-outs redrawn
- board text added: "Designed by Stephan Ahonen Revision 2025-07-20 Full schematics and other repair info at https://github.com/Solomute/STEVEannouncer"
- board text removed: "Designed by Stephan Ahonen Revision 2025-07-01 Full schematics and other repair info at https://github.com/Solomute/STEVEannouncer"
- board text removed: "Mechanical Keyboard Switches (i.e. Cherry MX)"
