File: PCB/IFBpath.kicad_sch (KiCad schematic)
At the start: 43 parts, among them J402 Conn_01x03, J403 Conn_01x03, J404 Conn_01x03, J405 Conn_01x03, J406 NRJ6HF, J407 NRJ6HF, U401 THAT2162, U402 OPA1678, U403 OPA1622

Commit message: Wooooooo
Parts:
- removed D405: BAS716, Diode_SMD:D_SOD-523, symbol Diode:1N4148WT
- added D406: BAS716, Diode_SMD:D_SOD-523, symbol Diode:1N4148WT
- added R410: 1Meg, Resistor_SMD:R_0402_1005Metric, symbol Device:R
- added R411: 10k, Resistor_SMD:R_0402_1005Metric, symbol Device:R
- added R412, R413: 330k, Resistor_SMD:R_0402_1005Metric, symbol Device:R
- C401, C402, C407: value 1u -> 1u/50V; footprint (none) -> Capacitor_SMD:C_0402_1005Metric; Mouser Part Number (none) -> 81-GRM155R61H105KE5D
- C405, C406, C410, C411, C412, C413, C414, C415: Mouser Part Number (none) -> 81-GRM155R62A104KE4D
- J402, J403, J404, J405: symbol Connector_Generic:Conn_01x03 -> STEVEannouncer:JST_B3B_PH
- J406, J407: symbol Connector_Audio:AudioJack3_Ground_Switch -> Connector_Audio:AudioJack3_Switch
- R405, R406: value 1Meg -> 80.6k
- R407: value 6.8k -> 80.6k
- RV401, RV402: footprint (none) -> STEVEannouncer:Pot
- U402: symbol Device:Opamp_Dual -> STEVEannouncer:OPA1678
- U403: footprint Package_SON:Texas_S-PVSON-N10 -> Package_SON:Texas_S-PVSON-N10_ThermalVias
Connections:
- net +5V: now also R405.1, R406.1, U402.8 (V+), D406.1 (K), R410.2; no longer U402.4 (V-), U403.8 (EN)
- net -5V: now also U402.4 (V-), U402.9 (Pad); no longer U402.8 (V+)
- net GND: now also R411.1; no longer J406.G, J407.G
- net at C405.1, J403.2 (Pin_2), U402.3 (+): now also R412.1; no longer R405.2
- net at C406.1, J404.2 (Pin_2), U402.5 (+): now also R413.2; no longer R406.2
- new net: J404.1 (Pin_1), R406.2
- new net: J403.1 (Pin_1), R405.2
- new net: C407.2, D406.2 (A), R410.1, U403.8 (EN)
- new net: R407.2, R411.2, R412.2, R413.1
Other:
- moved on the sheet: R407

Commit message: lalalalala
Parts:
- renumbered C408 to C407, C409 to C408, C407 to C409, D406 to D405, J404 to J403, J405 to J404, J403 to J405, R412 to R405, R413 to R406, R406 to R407, R405 to R408, R407 to R409, R411 to R410, R408 to R411, R409 to R412, R410 to R413

Commit message: progress
Connections:
- net GND: now also U403.1 (+), U403.5 (+)
- net at C408.1, R412.1: now also U401.15 (OUT), U403.6 (-); no longer U403.5 (+)
- net at C407.1, R411.1: now also U401.2 (OUT), U403.10 (-); no longer U403.1 (+)
- no-connect marks 0 -> 2
Other:
- moved on the sheet: C407, C408, R411, R412

Commit message: Moar Progress
Parts:
- J401: footprint Connector_Audio:Jack_XLR_Neutrik_NC3FAH2_Horizontal -> STEVEannouncer:NC3FAH2
- J406, J407: footprint Connector_Audio:Jack_6.35mm_Neutrik_NRJ6HF_Horizontal -> STEVEannouncer:NRJ6HF
Connections:
- no-connect marks 2 -> 6
Changed lines of the file:
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@@
 	)
 	(no_connect
+		(at 132.08 76.2)
+	)
+	(no_connect
 		(at 93.98 118.11)
 	)
+	(no_connect
+		(at 135.89 163.83)
+	)
+	(no_connect
+		(at 135.89 149.86)
+	)
+	(no_connect
+		(at 138.43 99.06)
+	)
 	(wire
 		(pts
@@
 			)
 		)
-		(property "Footprint" "Connector_Audio:Jack_6.35mm_Neutrik_NRJ6HF_Horizontal"
+		(property "Footprint" "STEVEannouncer:NRJ6HF"
 			(at 226.06 118.11 0)
 			(effects
@@
 			)
 		)
-		(property "Description" "Audio Jack, 3 Poles (Stereo / TRS), Switched Poles (Normalling)"
+		(property "Description" ""
 			(at 226.06 118.11 0)
 			(effects
@@
 			)
 		)
-		(property "Footprint" "Connector_Audio:Jack_6.35mm_Neutrik_NRJ6HF_Horizontal"
+		(property "Footprint" "STEVEannouncer:NRJ6HF"
 			(at 226.06 91.44 0)
 			(effects
@@
 			)
 		)
-		(property "Description" "Audio Jack, 3 Poles (Stereo / TRS), Switched Poles (Normalling)"
+		(property "Description" ""
 			(at 226.06 91.44 0)
 			(effects
@@
 			)
 		)
-		(property "Footprint" "Connector_Audio:Jack_XLR_Neutrik_NC3FAH2_Horizontal"
+		(property "Footprint" "STEVEannouncer:NC3FAH2"
 			(at 46.99 77.47 0)
 			(effects
@@
 			)
 		)
-		(property "Description" "XLR Connector, Male or Female, 3 Pins, Discrete Ground Pin"
+		(property "Description" ""
 			(at 46.99 77.47 0)
 			(effects

Commit message: Even more more progress
Parts:
- added C416, C417: 100p, Capacitor_SMD:C_0402_1005Metric, symbol Device:C
- added FB401, FB402: FerriteBead, Inductor_SMD:L_0402_1005Metric, symbol Device:FerriteBead
Connections:
- net GND: now also C416.2, C417.1
- net IFB_PIN2: now also FB401.2; no longer J401.2
- net VCA_OUTR: now reaches C408.1, R412.1, U401.15 (OUT), U403.6 (-)
- net HP_R: now reaches C408.2, J406.R, R412.2, U403.7
- net HP_L: now reaches C407.2, J406.T, J407.T, R411.2, U403.9
- net at J401.3: now also C417.2, FB402.1; no longer C402.1
- net VCA_OUTL: now reaches C407.1, R411.1, U401.2 (OUT), U403.10 (-)
- net VCA_INL: now reaches D401.2 (A), D403.1 (K), R401.2, R403.1, U401.7 (IN)
- net VCA_INR: now reaches D402.2 (A), D404.1 (K), R402.2, R404.1, U401.10 (IN)
- net VCAL_E-: now reaches U401.4 (E-), U402.1, U402.2 (-)
- net VCAR_E-: now reaches U401.13 (E-), U402.6 (-), U402.7
- new net: C416.1, FB401.1, J401.2
- new net IFB_Pin3: C402.1, FB402.2
Other:
- moved on the sheet: J401

Commit message: Yeet
Parts:
- B401, B402: value ~ -> Plastic Nut
- J401: value ~ -> NC3FAH2
Changed lines of the file:
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@@
 			)
 		)
-		(property "Value" "~"
+		(property "Value" "Plastic Nut"
 			(at 255.27 118.11 0)
 			(effects
@@
 			)
 		)
-		(property "Value" "~"
+		(property "Value" "NC3FAH2"
 			(at 34.29 69.85 0)
 			(effects
@@
 			)
 		)
-		(property "Value" "~"
+		(property "Value" "Plastic Nut"
 			(at 255.27 90.17 0)
 			(effects

Commit message: I think I can fab this????
Parts:
- U402: footprint Package_SON:WSON-8-1EP_3x3mm_P0.5mm_EP1.2x2mm_ThermalVias -> STEVEannouncer:WSON-8-1EP_3x3mm_P0.5mm_EP1.2x2mm_ThermalVias
- U403: footprint Package_SON:Texas_S-PVSON-N10_ThermalVias -> STEVEannouncer:OPA1622
Changed lines of the file:
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@@
 			)
 		)
-		(property "Footprint" "Package_SON:Texas_S-PVSON-N10_ThermalVias"
+		(property "Footprint" "STEVEannouncer:OPA1622"
 			(at 161.29 133.35 0)
 			(effects
@@
 			)
 		)
-		(property "Datasheet" "http://www.ti.com/lit/ds/symlink/opa1622.pdf"
+		(property "Datasheet" ""
 			(at 161.29 123.19 0)
 			(effects
@@
 			)
 		)
-		(property "Description" "High-Fidelity, Bipolar-Input, Audio Operational Amplifier, VSON-10"
+		(property "Description" ""
 			(at 161.29 123.19 0)
 			(effects
@@
 			)
 		)
-		(property "Footprint" "Package_SON:Texas_S-PVSON-N10_ThermalVias"
+		(property "Footprint" "STEVEannouncer:OPA1622"
 			(at 161.29 85.09 0)
 			(effects
@@
 			)
 		)
-		(property "Datasheet" "http://www.ti.com/lit/ds/symlink/opa1622.pdf"
+		(property "Datasheet" ""
 			(at 161.29 74.93 0)
 			(effects
@@
 			)
 		)
-		(property "Description" "High-Fidelity, Bipolar-Input, Audio Operational Amplifier, VSON-10"
+		(property "Description" ""
 			(at 161.29 74.93 0)
 			(effects
@@
 			)
 		)
-		(property "Footprint" "Package_SON:Texas_S-PVSON-N10_ThermalVias"
+		(property "Footprint" "STEVEannouncer:OPA1622"
 			(at 270.51 43.18 0)
 			(effects
@@
 			)
 		)
-		(property "Datasheet" "http://www.ti.com/lit/ds/symlink/opa1622.pdf"
+		(property "Datasheet" ""
 			(at 270.51 33.02 0)
 			(effects
@@
 			)
 		)
-		(property "Description" "High-Fidelity, Bipolar-Input, Audio Operational Amplifier, VSON-10"
+		(property "Description" ""
 			(at 270.51 33.02 0)
 			(effects
@@
 			)
 		)
-		(property "Footprint" "Package_SON:WSON-8-1EP_3x3mm_P0.5mm_EP1.2x2mm_ThermalVias"
+		(property "Footprint" "STEVEannouncer:WSON-8-1EP_3x3mm_P0.5mm_EP1.2x2mm_ThermalVias"
 			(at 232.41 33.02 0)
 			(effects
@@
 			)
 		)
-		(property "Footprint" "Package_SON:WSON-8-1EP_3x3mm_P0.5mm_EP1.2x2mm_ThermalVias"
+		(property "Footprint" "STEVEannouncer:WSON-8-1EP_3x3mm_P0.5mm_EP1.2x2mm_ThermalVias"
 			(at 106.68 144.78 0)
 			(effects
@@
 			)
 		)
-		(property "Footprint" "Package_SON:WSON-8-1EP_3x3mm_P0.5mm_EP1.2x2mm_ThermalVias"
+		(property "Footprint" "STEVEannouncer:WSON-8-1EP_3x3mm_P0.5mm_EP1.2x2mm_ThermalVias"
 			(at 106.68 93.98 0)
 			(effects

Commit message: Enclosure files
Parts:
- C403, C404, C407, C408, C416, C417: Mouser Part Number (none) -> 791-0402N101K160CT
- J401: Mouser Part Number (none) -> 568-NC3FAH-2
- R401, R402, R411, R412: Mouser Part Number (none) -> 603-RC0402FR-1320KL
- R403, R404: Mouser Part Number (none) -> 652-CR0402FX-6801GLF
- R405, R406: Mouser Part Number (none) -> 603-RC0402FR-13330KL
- R407, R408, R409: Mouser Part Number (none) -> 652-CR0402-FX8062GLF
- R410: Mouser Part Number (none) -> 652-CR0402FX-1002GLF
- R413: Mouser Part Number (none) -> 603-RC0402FR-7W1ML
Changed lines of the file:
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@@
 			)
 		)
+		(property "Mouser Part Number" "603-RC0402FR-1320KL"
+			(at 162.56 140.97 90)
+			(effects
+				(font
+					(size 1.27 1.27)
+				)
+				(hide yes)
+			)
+		)
 		(pin "2"
 		)
@@
 			)
 		)
+		(property "Mouser Part Number" "603-RC0402FR-1320KL"
+			(at 161.29 92.71 90)
+			(effects
+				(font
+					(size 1.27 1.27)
+				)
+				(hide yes)
+			)
+		)
 		(pin "2"
 		)
@@
 			)
 		)
+		(property "Mouser Part Number" "603-RC0402FR-1320KL"
+			(at 71.12 77.47 90)
+			(effects
+				(font
+					(size 1.27 1.27)
+				)
+				(hide yes)
+			)
+		)
 		(pin "2"
 		)
@@
 			)
 		)
+		(property "Mouser Part Number" "791-0402N101K160CT"
+			(at 43.18 106.68 0)
+			(effects
+				(font
+					(size 1.27 1.27)
+				)
+				(hide yes)
+			)
+		)
 		(pin "1"
 		)
@@
 			)
 		)
+		(property "Mouser Part Number" "791-0402N101K160CT"
+			(at 162.56 130.81 90)
+			(effects
+				(font
+					(size 1.27 1.27)
+				)
+				(hide yes)
+			)
+		)
 		(pin "2"
 		)
@@
 			)
 		)
+		(property "Mouser Part Number" "652-CR0402FX-6801GLF"
+			(at 80.01 132.08 0)
+			(effects
+				(font
+					(size 1.27 1.27)
+				)
+				(hide yes)
+			)
+		)
 		(pin "1"
 		)
@@
 			)
 		)
+		(property "Mouser Part Number" "791-0402N101K160CT"
+			(at 161.29 82.55 90)
+			(effects
+				(font
+					(size 1.27 1.27)
+				)
+				(hide yes)
+			)
+		)
 		(pin "2"
 		)
@@
 			)
 		)
+		(property "Mouser Part Number" "603-RC0402FR-1320KL"
+			(at 71.12 125.73 90)
+			(effects
+				(font
+					(size 1.27 1.27)
+				)
+				(hide yes)
+			)
+		)
 		(pin "2"
 		)
@@
 			)
 		)
+		(property "Mouser Part Number" "603-RC0402FR-13330KL"
+			(at 119.38 116.84 0)
+			(effects
+				(font
+					(size 1.27 1.27)
+				)
+				(hide yes)
+			)
+		)
 		(pin "1"
 		)
@@
 			)
 		)
+		(property "Mouser Part Number" "652-CR0402FX-6801GLF"
+			(at 80.01 85.09 0)
+			(effects
+				(font
+					(size 1.27 1.27)
+				)
+				(hide yes)
+			)
+		)
 		(pin "1"
 		)
@@
 			)
 		)
+		(property "Mouser Part Number" "791-0402N101K160CT"
+			(at 80.01 140.97 0)
+			(effects
+				(font
+					(size 1.27 1.27)
+				)
+				(hide yes)
+			)
+		)
 		(pin "2"
 		)
@@
 			)
 		)
+		(property "Mouser Part Number" "652-CR0402-FX8062GLF"
+			(at 142.24 105.41 0)
+			(effects
+				(font
+					(size 1.27 1.27)
+				)
+				(hide yes)
+			)
+		)
 		(pin "2"
 		)
@@
 			)
 		)
+		(property "Mouser Part Number" "652-CR0402-FX8062GLF"
+			(at 129.54 88.9 90)
+			(effects
+				(font
+					(size 1.27 1.27)
+				)
+				(hide yes)
+			)
+		)
 		(pin "2"
 		)
@@
 			)
 		)
+		(property "Mouser Part Number" "791-0402N101K160CT"
+			(at 80.01 93.98 0)
+			(effects
+				(font
+					(size 1.27 1.27)
+				)
+				(hide yes)
+			)
+		)
 		(pin "2"
 		)
@@
 			)
 		)
+		(property "Mouser Part Number" "791-0402N101K160CT"
+			(at 43.18 99.06 0)
+			(effects
+				(font
+					(size 1.27 1.27)
+				)
+				(hide yes)
+			)
+		)
 		(pin "1"
 		)
@@
 			)
 		)
+		(property "Mouser Part Number" "568-NC3FAH-2"
+			(at 34.29 77.47 0)
+			(effects
+				(font
+					(size 1.27 1.27)
+				)
+				(hide yes)
+			)
+		)
 		(pin "3"
 		)
@@
 			)
 		)
+		(property "Mouser Part Number" "603-RC0402FR-7W1ML"
+			(at 181.61 57.15 0)
+			(effects
+				(font
+					(size 1.27 1.27)
+				)
+				(hide yes)
+			)
+		)
 		(pin "2"
 		)
@@
 			)
 		)
+		(property "Mouser Part Number" "603-RC0402FR-13330KL"
+			(at 119.38 101.6 0)
+			(effects
+				(font
+					(size 1.27 1.27)
+				)
+				(hide yes)
+			)
+		)
 		(pin "1"
 		)
@@
 			)
 		)
+		(property "Mouser Part Number" "652-CR0402-FX8062GLF"
+			(at 128.27 134.62 0)
+			(effects
+				(font
+					(size 1.27 1.27)
+				)
+				(hide yes)
+			)
+		)
 		(pin "2"
 		)
@@
 			(at 142.24 113.03 0)
 			(effects
+				(font
+					(size 1.27 1.27)
+				)
+				(hide yes)
+			)
+		)
+		(property "Mouser Part Number" "652-CR0402FX-1002GLF"
+			(at 142.24 113.03 0)
+			(effects
