File: PCB/MicPath.kicad_sch (KiCad schematic)
At the start: 53 parts, among them J301 NC3FAH, J302 Conn_01x02, J303 Conn_01x02, J304 Conn_01x02, J305 Conn_01x02, J306 NC3MAH, J307 NC3MAH, SW301 SW_SPST, SW302 SW_SPST, U301 THAT1512, U302 TMUX6236, U303 THAT1646, U304 THAT1646

Commit message: Wooooooo
Parts:
- removed U303: THAT1646, Package_SO:SO-8_3.9x4.9mm_P1.27mm, symbol STEVEannouncer:THAT1646
- added D308: BAS716, Diode_SMD:D_SOD-523, symbol Diode:1N4148WT
- added R309, R313, R315, R319, R320: 20k, Resistor_SMD:R_0402_1005Metric, symbol Device:R
- added R310, R312, R316, R317: 1k, Resistor_SMD:R_0402_1005Metric, symbol Device:R
- added R311, R318: 100, Resistor_SMD:R_0402_1005Metric, symbol Device:R
- added R314: 10k, Resistor_SMD:R_0402_1005Metric, symbol Device:R
- added U303: OPA1678, Package_SON:WSON-8-1EP_3x3mm_P0.5mm_EP1.2x2mm_ThermalVias, symbol STEVEannouncer:OPA1678
- C304, C305: footprint (none) -> Capacitor_SMD:CP_Elec_6.3x7.7; Mouser Part Number (none) -> 647-UCD1J220MCL1GS
- C306: footprint (none) -> Capacitor_SMD:C_1206_3216Metric; Mouser Part Number (none) -> 81-GRM31CR60J107KE8L
- C307, C308, C309, C310, C311, C312, C313: Mouser Part Number (none) -> 81-GRM155R62A104KE4D
- C314, C315: value 10u -> 100n; footprint (none) -> Capacitor_SMD:C_0402_1005Metric; Mouser Part Number (none) -> 81-GRM155R62A104KE4D
- C316, C317: footprint (none) -> Capacitor_SMD:C_0603_1608Metric; Mouser Part Number (none) -> 187-CL10A106KP8NNWC
- J302, J303, J304, J305: symbol Connector_Generic:Conn_01x02 -> STEVEannouncer:JST_B2B_PH
Connections:
- net +5V: now also U303.8 (V+)
- net -5V: now also R319.2, R320.2, U303.4 (V-), U303.9 (Pad)
- net GND: now also C314.1, C315.1, U302.12 (SB), U302.2 (SA), U302.6 (GND)
- net at J304.2 (Pin_2), U302.9 (SEL): now also D308.2 (A), R319.1
- net at J302.2 (Pin_2), U302.1 (SEL): now also D308.1 (K), R320.1
- net at D306.3, FB302.1: now also R317.1, R318.2; no longer C315.2
- net at U302.10 (SA): now also U301.6 (Out), U302.4 (SB)
- net at D306.2, FB301.1: now also R310.1, R311.2; no longer C314.2
- net at U302.11 (D): now also R309.1, R314.1; no longer U302.4 (SB)
- net at U304.4 (IN): now also U302.3 (D); no longer U302.12 (SB)
- new net: R315.2, R317.2, U303.5 (+)
- new net: R314.2, R316.2, U303.6 (-)
- new net: R316.1, R318.1, U303.7
- new net: C315.2, R315.1
- new net: R311.1, R312.1, U303.1
- new net: R312.2, R313.2, U303.2 (-)
- new net: R309.2, R310.2, U303.3 (+)
- new net: C314.2, R313.1
Other:
- moved on the sheet: C301, C302, C303, C304, C305, C306, C307, C308, C309, C310, C311, C312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

Commit message: lalalalala
Parts:
- R307: renamed from R308; value 20k -> 330k
- R308: renamed from R307; value 20k -> 330k
- R309: renamed from R320; value 20k -> 330k
- R310: renamed from R319; value 20k -> 330k
- renumbered C309 to C301, C301 to C302, C302 to C303, C303 to C304, C304 to C305, C305 to C306, C306 to C307, C310 to C308, C311 to C309, C307 to C310, C308 to C311, C314 to C312, C315 to C313, C312 to C314, C313 to C315, C320 to C318, C321 to C319, C318 to C320, C319 to C321, D304 to D302, D305 to D303, D302 to D304, D303 to D305, D308 to D306, D306 to D308, FB303 to FB301, FB304 to FB302, FB301 to FB303, FB302 to FB304, J303 to J302, J304 to J303, J302 to J304, R309 to R311, R314 to R312, R315 to R314, R310 to R315, R312 to R316, R316 to R317, R317 to R318, R311 to R319, R318 to R320, U302 to U301, U303 to U302, U301 to U303
Connections:
- net Micpre+: now reaches D301.2, D304.1 (K), R301.1, R303.1, U303.3 (+In)
- net MicOut-: now reaches C317.2, D307.3, FB302.1, U304.1 (OUT-)
- net Mic3: now reaches C304.2, C306.1, J301.3
- net MicOut3: now reaches C319.2, FB302.2, J307.3
- net MicOut+: now reaches C316.2, D307.2, FB301.1, U304.8 (OUT+)
- net MicOut2: now reaches C318.1, FB301.2, J307.2
- net Mic2: now reaches C303.1, C305.1, J301.2
- net RG2: now reaches C307.2, D305.2 (A), U303.8 (Rg2)
- net Micpre-: now reaches D301.3, D305.1 (K), R302.1, R304.2, U303.2 (-In)
- net MicpreOut: now reaches U301.10 (SA), U301.4 (SB), U303.6 (Out)
- net MicOut: now reaches U301.3 (D), U304.4 (IN)
- net RG1: now reaches D304.2 (A), R306.2, U303.1 (Rg1)
Other:
- moved on the sheet: C308

Commit message: progress
Parts:
- added C322: 100n, Capacitor_SMD:C_0402_1005Metric, symbol Device:C
- R312: value 10k -> 20k
Connections:
- net +5V: now also U301.13 (VCC), C322.1; no longer C301.2, U301.5 (VSS)
- net -5V: now also U301.5 (VSS); no longer U301.13 (VCC)
- net GND: now also C301.2, C322.2
- net MicOut+: now also D307.3; no longer D307.2
- net MicOut-: now also D307.2; no longer D307.3
- net Micpre+: now also D301.3; no longer D301.2
- net Micpre-: now also D301.2; no longer D301.3
- net TBSel: now reaches D306.2 (A), J303.2 (Pin_2), R310.1, U301.9 (SEL)
- net MuteSel: now reaches D306.1 (K), J304.2 (Pin_2), R309.1, U301.1 (SEL)
- net TBOut: now reaches R311.1, R312.1, U301.11 (D)
Other:
- moved on the sheet: C301, U301C

Commit message: Moar Progress
Parts:
- J301: footprint Connector_Audio:Jack_XLR_Neutrik_NC3FAH2_Horizontal -> STEVEannouncer:NC3FAH2
- J306, J307: footprint Connector_Audio:Jack_XLR_Neutrik_NC3MAH_Horizontal -> STEVEannouncer:NC3MAH
- SW301, SW302: footprint Button_Switch_Keyboard:SW_Cherry_MX_1.00u_PCB -> STEVEannouncer:CherrySwitch
Connections:
- no-connect marks 0 -> 4
Changed lines of the file:
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@@
 		(color 0 0 0 0)
 	)
+	(no_connect
+		(at 153.67 118.11)
+	)
+	(no_connect
+		(at 144.78 81.28)
+	)
+	(no_connect
+		(at 153.67 165.1)
+	)
+	(no_connect
+		(at 170.18 81.28)
+	)
 	(wire
 		(pts
@@
 			)
 		)
-		(property "Footprint" "Button_Switch_Keyboard:SW_Cherry_MX_1.00u_PCB"
+		(property "Footprint" "STEVEannouncer:CherrySwitch"
 			(at 163.83 72.39 0)
 			(effects
@@
 			)
 		)
-		(property "Description" "Single Pole Single Throw (SPST) switch"
+		(property "Description" ""
 			(at 163.83 72.39 0)
 			(effects
@@
 			)
 		)
-		(property "Footprint" "Connector_Audio:Jack_XLR_Neutrik_NC3FAH2_Horizontal"
+		(property "Footprint" "STEVEannouncer:NC3FAH2"
 			(at 25.4 125.73 0)
 			(effects
@@
 			)
 		)
-		(property "Description" "XLR Connector, Male or Female, 3 Pins, Discrete Ground Pin"
+		(property "Description" ""
 			(at 25.4 125.73 0)
 			(effects
@@
 			)
 		)
-		(property "Footprint" "Connector_Audio:Jack_XLR_Neutrik_NC3MAH_Horizontal"
+		(property "Footprint" "STEVEannouncer:NC3MAH"
 			(at 269.24 43.18 0)
 			(effects
@@
 			)
 		)
-		(property "Description" "XLR Connector, Male or Female, 3 Pins, Discrete Ground Pin"
+		(property "Description" ""
 			(at 269.24 43.18 0)
 			(effects
@@
 			)
 		)
-		(property "Footprint" "Button_Switch_Keyboard:SW_Cherry_MX_1.00u_PCB"
+		(property "Footprint" "STEVEannouncer:CherrySwitch"
 			(at 138.43 72.39 0)
 			(effects
@@
 			)
 		)
-		(property "Description" "Single Pole Single Throw (SPST) switch"
+		(property "Description" ""
 			(at 138.43 72.39 0)
 			(effects
@@
 			)
 		)
-		(property "Footprint" "Connector_Audio:Jack_XLR_Neutrik_NC3MAH_Horizontal"
+		(property "Footprint" "STEVEannouncer:NC3MAH"
 			(at 269.24 140.97 0)
 			(effects
@@
 			)
 		)
-		(property "Description" "XLR Connector, Male or Female, 3 Pins, Discrete Ground Pin"
+		(property "Description" ""
 			(at 269.24 140.97 0)
 			(effects

Commit message: Even more more progress
Parts:
- added C323, C324: 100n, Capacitor_SMD:C_0402_1005Metric, symbol Device:C
Connections:
- net GND: now also C323.1, C324.1
- net MuteSel: now also C324.2
- net TBSel: now also C323.2
- net TB_OUT2: now reaches C320.1, FB303.2, J306.2
- net TB_OUT3: now reaches C321.2, FB304.2, J306.3

Commit message: I think I can fab this????
Parts:
- J301: value NC3FAH -> NC3FAH2
- U302: footprint Package_SON:WSON-8-1EP_3x3mm_P0.5mm_EP1.2x2mm_ThermalVias -> STEVEannouncer:WSON-8-1EP_3x3mm_P0.5mm_EP1.2x2mm_ThermalVias
- U304: Mouser Part Number 887-THAT1646W16-U -> 887-1646S08-U
Connections:
- net -5V: no longer R309.2, R310.2
- net GND: now also R309.2, R310.2
Changed lines of the file:
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@@
 	)
 	(symbol
+		(lib_id "power:GND")
+		(at 167.64 152.4 180)
+		(unit 1)
+		(exclude_from_sim no)
+		(in_bom yes)
+		(on_board yes)
+		(dnp no)
+		(fields_autoplaced yes)
+		(property "Reference" "#PWR0325"
+			(at 167.64 146.05 0)
+			(effects
+				(font
+					(size 1.27 1.27)
+				)
+				(hide yes)
+			)
+		)
+		(property "Value" "GND"
+			(at 167.64 147.4753 0)
+			(effects
+				(font
+					(size 1.27 1.27)
+				)
+			)
+		)
+		(property "Footprint" ""
+			(at 167.64 152.4 0)
+			(effects
+				(font
+					(size 1.27 1.27)
+				)
+				(hide yes)
+			)
+		)
+		(property "Datasheet" ""
+			(at 167.64 152.4 0)
+			(effects
+				(font
+					(size 1.27 1.27)
+				)
+				(hide yes)
+			)
+		)
+		(property "Description" "Power symbol creates a global label with name \"GND\" , ground"
+			(at 167.64 152.4 0)
+			(effects
+				(font
+					(size 1.27 1.27)
+				)
+				(hide yes)
+			)
+		)
+		(pin "1"
+		)
+		(instances
+			(project "STEVEannouncer"
+				(path "/1a37937a-d840-40ca-a420-44780efca6fe/ed5acf0b-c0f0-4ec2-837f-fd4292e4b1bc"
+					(reference "#PWR0325")
+					(unit 1)
+				)
+			)
+		)
+	)
+	(symbol
 		(lib_id "Device:C")
 		(at 256.54 46.99 0)
@@
 			)
 		)
-		(property "Footprint" "Package_SON:WSON-8-1EP_3x3mm_P0.5mm_EP1.2x2mm_ThermalVias"
+		(property "Footprint" "STEVEannouncer:WSON-8-1EP_3x3mm_P0.5mm_EP1.2x2mm_ThermalVias"
 			(at 104.14 40.64 0)
 			(effects
@@
 			)
 		)
-		(property "Footprint" "Package_SON:WSON-8-1EP_3x3mm_P0.5mm_EP1.2x2mm_ThermalVias"
+		(property "Footprint" "STEVEannouncer:WSON-8-1EP_3x3mm_P0.5mm_EP1.2x2mm_ThermalVias"
 			(at 207.01 35.56 0)
 			(effects
@@
 			)
 		)
-		(property "Footprint" "Package_SON:WSON-8-1EP_3x3mm_P0.5mm_EP1.2x2mm_ThermalVias"
+		(property "Footprint" "STEVEannouncer:WSON-8-1EP_3x3mm_P0.5mm_EP1.2x2mm_ThermalVias"
 			(at 207.01 83.82 0)
 			(effects
@@
 			)
 		)
-		(property "Value" "NC3FAH"
+		(property "Value" "NC3FAH2"
 			(at 25.4 118.11 0)
 			(effects
@@
 	)
 	(symbol
-		(lib_id "power:-5V")
-		(at 167.64 152.4 0)
-		(unit 1)
-		(exclude_from_sim no)
-		(in_bom yes)
-		(on_board yes)
-		(dnp no)
-		(fields_autoplaced yes)
-		(property "Reference" "#PWR0325"
-			(at 167.64 156.21 0)
-			(effects
-				(font
-					(size 1.27 1.27)
-				)
-				(hide yes)
-			)
-		)
-		(property "Value" "-5V"
-			(at 167.64 147.32 0)
-			(effects
-				(font
-					(size 1.27 1.27)
-				)
-			)
-		)
-		(property "Footprint" ""
-			(at 167.64 152.4 0)
-			(effects
-				(font
-					(size 1.27 1.27)
-				)
-				(hide yes)
-			)
-		)
-		(property "Datasheet" ""
-			(at 167.64 152.4 0)
-			(effects
-				(font
-					(size 1.27 1.27)
-				)
-				(hide yes)
-			)
-		)
-		(property "Description" "Power symbol creates a global label with name \"-5V\""
-			(at 167.64 152.4 0)
-			(effects
-				(font
-					(size 1.27 1.27)
-				)
-				(hide yes)
-			)
-		)
-		(pin "1"
-		)
-		(instances
-			(project "STEVEannouncer"
-				(path "/1a37937a-d840-40ca-a420-44780efca6fe/ed5acf0b-c0f0-4ec2-837f-fd4292e4b1bc"
-					(reference "#PWR0325")
-					(unit 1)
-				)
-			)
-		)
-	)
-	(symbol
 		(lib_id "Device:C")
 		(at 213.36 133.35 90)
@@
 	)
 	(symbol
+		(lib_id "power:GND")
+		(at 170.18 105.41 180)
+		(unit 1)
+		(exclude_from_sim no)
+		(in_bom yes)
+		(on_board yes)
+		(dnp no)
+		(fields_autoplaced yes)
+		(property "Reference" "#PWR0326"
+			(at 170.18 99.06 0)
+			(effects
+				(font
+					(size 1.27 1.27)
+				)
+				(hide yes)
+			)
+		)
+		(property "Value" "GND"
+			(at 170.18 100.33 0)
+			(effects
+				(font
+					(size 1.27 1.27)
+				)
+			)
+		)
+		(property "Footprint" ""
+			(at 170.18 105.41 0)
+			(effects
+				(font
+					(size 1.27 1.27)
+				)
+				(hide yes)
+			)
+		)
+		(property "Datasheet" ""
+			(at 170.18 105.41 0)
+			(effects
+				(font
+					(size 1.27 1.27)
+				)
+				(hide yes)
+			)
+		)
+		(property "Description" "Power symbol creates a global label with name \"GND\" , ground"
+			(at 170.18 105.41 0)
+			(effects
+				(font
+					(size 1.27 1.27)
+				)
+				(hide yes)
+			)
+		)
+		(pin "1"
+		)
+		(instances
+			(project "STEVEannouncer"
+				(path "/1a37937a-d840-40ca-a420-44780efca6fe/ed5acf0b-c0f0-4ec2-837f-fd4292e4b1bc"
+					(reference "#PWR0326")
+					(unit 1)
+				)
+			)
+		)
+	)
+	(symbol
 		(lib_id "STEVEannouncer:JST_B2B_PH")
 		(at 137.16 81.28 90)
@@
 			)
 		)
-		(property "Mouser Part Number" "887-THAT1646W16-U"
+		(property "Mouser Part Number" "887-1646S08-U"
 			(at 208.28 142.24 0)
 			(effects
@@
 					(unit 1)
 				)
-			)
-		)
-	)
-	(symbol
-		(lib_id "power:-5V")
-		(at 170.18 105.41 0)
-		(unit 1)
-		(exclude_from_sim no)
-		(in_bom yes)
-		(on_board yes)
-		(dnp no)
-		(fields_autoplaced yes)
-		(property "Reference" "#PWR0326"
-			(at 170.18 109.22 0)
-			(effects
-				(font
-					(size 1.27 1.27)
-				)
-				(hide yes)
-			)
-		)
-		(property "Value" "-5V"
-			(at 170.18 100.33 0)
-			(effects
-				(font
-					(size 1.27 1.27)
-				)
-			)
-		)
-		(property "Footprint" ""
-			(at 170.18 105.41 0)
-			(effects
-				(font
-					(size 1.27 1.27)
-				)
-				(hide yes)
-			)
-		)
-		(property "Datasheet" ""
-			(at 170.18 105.41 0)
-			(effects
-				(font
-					(size 1.27 1.27)
-				)
-				(hide yes)
-			)
-		)
-		(property "Description" "Power symbol creates a global label with name \"-5V\""
-			(at 170.18 105.41 0)
-			(effects
-				(font
-					(size 1.27 1.27)
-				)
-				(hide yes)
-			)
-		)
-		(pin "1"
-		)
-		(instances
-			(project "STEVEannouncer"
-				(path "/1a37937a-d840-40ca-a420-44780efca6fe/ed5acf0b-c0f0-4ec2-837f-fd4292e4b1bc"
-					(reference "#PWR0326")
-					(unit 1)
-				)

Commit message: There, I ordered it
Parts:
- removed D306: BAS716, Diode_SMD:D_SOD-523, symbol Diode:1N4148WT
- added D306: D_Schottky, Diode_SMD:D_SOD-523, symbol Device:D_Schottky
- R307, R308: value 330k -> 20k
- SW301, SW302: footprint STEVEannouncer:CherrySwitch -> STEVEannouncer:SW_choc_v1_1u
Connections:
- net +5V: now also R309.2, R310.2; no longer R307.2, R308.2
- net GND: now also R307.2, R308.2, U301.10 (SA), U301.4 (SB); no longer R309.2, R310.2, U301.12 (SB), U301.2 (SA)
- net MicpreOut: now also U301.12 (SB), U301.2 (SA); no longer U301.10 (SA), U301.4 (SB)
- net MuteSel: now also D306.2 (A)
- net TBSel: now also D306.1 (K)
- net at SW302.1 (A): now also J305.2 (Pin_2); no longer J305.1 (Pin_1)
- net at SW302.2 (B): now also J305.1 (Pin_1); no longer J305.2 (Pin_2)
- net at SW301.1 (A): now also J302.2 (Pin_2); no longer J302.1 (Pin_1)
- net at SW301.2 (B): now also J302.1 (Pin_1); no longer J302.2 (Pin_2)
Other:
- moved on the sheet: R309, R310

Commit message: Enclosure files
Parts:
- C302, C318, C319, C320, C321: Mouser Part Number (none) -> 791-0402N101K160CT
- C303, C304: Mouser Part Number (none) -> 80-C0402C471K5R
- J301: Mouser Part Number (none) -> 568-NC3FAH-2
- J306, J307: Mouser Part Number (none) -> 568-NC3MAH
- R301, R302: Mouser Part Number (none) -> 652-CR1206-JW-100ELF
- R303, R304, R315, R316, R317, R318: Mouser Part Number (none) -> 708-RMCF0402FT1K00
- R305, R307, R308, R311, R312, R313, R314: Mouser Part Number (none) -> 603-RC0402FR-1320KL
- R306: Mouser Part Number (none) -> 708-RMCF0402FT270R
- R309, R310: Mouser Part Number (none) -> 603-RC0402FR-13330KL
- R319, R320: Mouser Part Number (none) -> 652-CR0402FX-1000GLF
