File: PCB/MicPath.kicad_sch (KiCad schematic)
At the start: 69 parts, among them J301 NC3FAH2, J302 Conn_01x02, J303 Conn_01x02, J304 Conn_01x02, J305 Conn_01x02, J306 NC3MAH, J307 NC3MAH, SW301 SW_SPST, SW302 SW_SPST, U301 TMUX6236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

Commit message: revisionnnnn
Parts:
- added C325, C326: 100n, Capacitor_SMD:C_0402_1005Metric, symbol Device:C
- added C327: 10u, Capacitor_SMD:C_0603_1608Metric, symbol Device:C
- added C328, C329: 470p, Capacitor_SMD:C_0402_1005Metric, symbol Device:C
- added R321, R322: 10k, Resistor_SMD:R_0402_1005Metric, symbol Device:R
- added U305: OPA202, Package_TO_SOT_SMD:SOT-23-5, symbol Amplifier_Operational:OPA196xDBV
- R306: value 270 -> 100
Connections:
- net +5V: now also C326.2, U305.5 (V+)
- net -5V: now also C325.2, U305.2 (V-)
- net GND: now also R314.1, C325.1, C326.1, C328.2, C329.2, R322.2; no longer C313.1, U303.5 (Ref)
- net MicOut: now also C328.1
- net MicpreOut: now also R321.1
- net TBOut: now also C313.2, C329.1; no longer R312.1
- new net: R322.1, U305.3 (+)
- new net: C313.1, R312.1
- new net: C327.1, R321.2, U305.4 (-)
- new net: C327.2, U303.5 (Ref), U305.1
Other:
- moved on the sheet: C313
