File: PCB/MicPath.kicad_sch (KiCad schematic)
At the start: 77 parts, among them J301 NC3FAH2, J302 Conn_01x02, J303 Conn_01x02, J304 Conn_01x02, J305 Conn_01x02, J306 NC3MAH, J307 NC3MAH, SW301 SW_SPST, SW302 SW_SPST, U301 TMUX6236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

Commit message: Rev 2025-07-20
Parts:
- removed J302, J305: Conn_01x02, Connector_JST:JST_PH_B2B-PH-SM4-TB_1x02-1MP_P2.00mm_Vertical, symbol STEVEannouncer:JST_B2B_PH
- added J302, J305: Conn_01x02, STEVEannouncer:SolderWire-0.15sqmm_1x02_P4mm_D0.5mm_OD1.5mm, symbol Connector_Generic:Conn_01x02
- C328, C329: Mouser Part Number (none) -> 80-C0402C471K5R
- D301, D307, D308: value BAS3007ARPPE6327HTSA1 -> BAS3007
- D302, D303: Gearlabs Part Number D-Zener-5V6-123-2 -> (none)
- R306: Mouser Part Number 708-RMCF0402FT270R -> 652-CR0402FX-1000GLF
- R321, R322: Mouser Part Number (none) -> 652-CR0402FX-1002GLF
- U302: Gearlabs Part Number EXT-OPA1678 -> (none)
- U305: Mouser Part Number (none) -> 595-OPA202IDBVR
Connections:
- net at SW302.1 (A): now also J305.1 (Pin_1)
- net at SW302.2 (B): now also J305.2 (Pin_2)
- net at SW301.1 (A): now also J302.1 (Pin_1)
- net at SW301.2 (B): now also J302.2 (Pin_2)
- no-connect marks 4 -> 2
Other:
- moved on the sheet: SW301, SW302

Commit message: Tidying up
Parts:
- U302: footprint STEVEannouncer:WSON-8-1EP_3x3mm_P0.5mm_EP1.2x2mm_ThermalVias -> Package_SON:WSON-8-1EP_3x3mm_P0.5mm_EP1.2x2mm_ThermalVias; Gearlabs Part Number (none) -> EXT-OPA1678
Other:
- note added: "Buttons"
- note added: "DC Offset Servo"
- note added: "Mic Preamp"
- note added: "Power/Bypassing"
- note added: "Routing"
- moved on the sheet: C302, C303, C304, C305, C306, C307, C310, C311, C323, C324, C325, C326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
