File: PCB/Power.kicad_sch (KiCad schematic)
At the start: 27 parts, among them J201 Barrel_Jack, Q201 BC847, Q202 BCV49, U201 LV3842, U202 LV3842

Commit message: Wooooooo
Parts:
- removed J201: Barrel_Jack, Connector_BarrelJack:BarrelJack_Horizontal, symbol Connector:Barrel_Jack
- removed R204: 20k, Resistor_SMD:R_0402_1005Metric, symbol Device:R
- added J202: Barrel_Jack_Switch, STEVEannouncer:Barrel Jack, symbol Connector:Barrel_Jack_Switch
- C201: value 100u -> 1u/50V; footprint (none) -> Capacitor_SMD:C_0402_1005Metric; Mouser Part Number (none) -> 81-GRM155R61H105KE5D
- C203, C204: footprint (none) -> Capacitor_SMD:C_0603_1608Metric; Mouser Part Number (none) -> 81-GRT188R61H225KE3D
- C205, C206: Mouser Part Number (none) -> 81-GRM155R62A104KE4D
- C207, C208: footprint (none) -> Capacitor_SMD:C_1206_3216Metric; Mouser Part Number (none) -> 791-1206X226K100CT
Connections:
- net GND: now also J202.2, J202.3
- net at C201.2: now also D202.2 (A), Q201.2 (E), R202.2, R205.2
- net at D203.2 (A): now also J202.1
Other:
- moved on the sheet: C201

Commit message: lalalalala
Parts:
- renumbered J202 to J201, R205 to R204, R206 to R205, R207 to R206, R208 to R207, R209 to R208
Changed lines of the file:
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@@
 		(on_board yes)
 		(dnp no)
-		(property "Reference" "R206"
+		(property "Reference" "R205"
 			(at 209.55 110.4899 0)
 			(effects
@@
 			(project ""
 				(path "/1a37937a-d840-40ca-a420-44780efca6fe/eebf1098-e67c-4d58-86f4-2b87a99f6ef8"
-					(reference "R206")
+					(reference "R205")
 					(unit 1)
 				)
@@
 		(on_board yes)
 		(dnp no)
-		(property "Reference" "R207"
+		(property "Reference" "R206"
 			(at 209.55 143.5099 0)
 			(effects
@@
 			(project "STEVEannouncer"
 				(path "/1a37937a-d840-40ca-a420-44780efca6fe/eebf1098-e67c-4d58-86f4-2b87a99f6ef8"
-					(reference "R207")
+					(reference "R206")
 					(unit 1)
 				)
@@
 		(dnp no)
 		(fields_autoplaced yes)
-		(property "Reference" "J202"
+		(property "Reference" "J201"
 			(at 95.25 109.22 0)
 			(effects
@@
 			(project ""
 				(path "/1a37937a-d840-40ca-a420-44780efca6fe/eebf1098-e67c-4d58-86f4-2b87a99f6ef8"
-					(reference "J202")
+					(reference "J201")
 					(unit 1)
 				)
@@
 		(on_board yes)
 		(dnp no)
-		(property "Reference" "R209"
+		(property "Reference" "R208"
 			(at 220.98 146.05 90)
 			(effects
@@
 			(project "STEVEannouncer"
 				(path "/1a37937a-d840-40ca-a420-44780efca6fe/eebf1098-e67c-4d58-86f4-2b87a99f6ef8"
-					(reference "R209")
+					(reference "R208")
 					(unit 1)
 				)
@@
 		(dnp no)
 		(fields_autoplaced yes)
-		(property "Reference" "R205"
+		(property "Reference" "R204"
 			(at 104.14 92.7099 0)
 			(effects
@@
 			(project "STEVEannouncer"
 				(path "/1a37937a-d840-40ca-a420-44780efca6fe/eebf1098-e67c-4d58-86f4-2b87a99f6ef8"
-					(reference "R205")
+					(reference "R204")
 					(unit 1)
 				)
@@
 		(on_board yes)
 		(dnp no)
-		(property "Reference" "R208"
+		(property "Reference" "R207"
 			(at 220.98 113.03 90)
 			(effects
@@
 			(project ""
 				(path "/1a37937a-d840-40ca-a420-44780efca6fe/eebf1098-e67c-4d58-86f4-2b87a99f6ef8"
-					(reference "R208")
-					(unit 1)
-				)
+					(reference "R207")
+					(unit 1)
+				)

Commit message: progress
Parts:
- added C209: 100n, Capacitor_SMD:C_0402_1005Metric, symbol Device:C
Connections:
- net -5V: now also C209.1
- net vbulk: now reaches C202.1, C203.1, C204.1, D202.1 (K), D203.1 (K), U201.4 (EN), U201.5 (VIN), U202.4 (EN), U202.5 (VIN)
- net vbulk: now also C209.2
Other:
- moved on the sheet: C204
Changed lines of the file:
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@@
 	)
 	(junction
+		(at 184.15 134.62)
+		(diameter 0)
+		(color 0 0 0 0)
+	)
+	(junction
 		(at 228.6 106.68)
 		(diameter 0)
@@
 	)
 	(junction
-		(at 182.88 134.62)
-		(diameter 0)
-		(color 0 0 0 0)
-	)
-	(junction
 		(at 90.17 73.66)
 		(diameter 0)
@@
 	)
 	(junction
+		(at 171.45 134.62)
+		(diameter 0)
+		(color 0 0 0 0)
+	)
+	(junction
 		(at 167.64 101.6)
 		(diameter 0)
@@
 	(wire
 		(pts
-			(xy 182.88 143.51) (xy 182.88 144.78)
+			(xy 171.45 143.51) (xy 171.45 144.78)
 		)
 		(stroke
@@
 	(wire
 		(pts
+			(xy 171.45 134.62) (xy 184.15 134.62)
+		)
+		(stroke
+			(width 0)
+			(type default)
+		)
+	)
+	(wire
+		(pts
 			(xy 58.42 73.66) (xy 58.42 67.31)
 		)
@@
 	(wire
 		(pts
-			(xy 182.88 134.62) (xy 182.88 135.89)
+			(xy 171.45 134.62) (xy 171.45 135.89)
 		)
 		(stroke
@@
 	(wire
 		(pts
-			(xy 167.64 134.62) (xy 182.88 134.62)
+			(xy 167.64 134.62) (xy 171.45 134.62)
 		)
 		(stroke
@@
 	(wire
 		(pts
-			(xy 182.88 134.62) (xy 190.5 134.62)
+			(xy 184.15 134.62) (xy 190.5 134.62)
 		)
 		(stroke
@@
 		)
 	)
+	(label "vbulk"
+		(at 152.4 101.6 0)
+		(effects
+			(font
+				(size 1.27 1.27)
+			)
+			(justify left bottom)
+		)
+	)
 	(global_label "IFB_PIN2"
 		(shape input)
@@
 	(symbol
 		(lib_id "Device:C")
-		(at 182.88 139.7 0)
+		(at 171.45 139.7 0)
 		(mirror y)
 		(unit 1)
@@
 		(dnp no)
 		(property "Reference" "C204"
-			(at 179.07 138.4299 0)
+			(at 167.64 138.4299 0)
 			(effects
 				(font
@@
 		)
 		(property "Value" "2.2u"
-			(at 179.07 140.9699 0)
+			(at 167.64 140.9699 0)
 			(effects
 				(font
@@
 		)
 		(property "Footprint" "Capacitor_SMD:C_0603_1608Metric"
-			(at 181.9148 143.51 0)
+			(at 170.4848 143.51 0)
 			(effects
 				(font
@@
 		)
 		(property "Datasheet" "~"
-			(at 182.88 139.7 0)
+			(at 171.45 139.7 0)
 			(effects
 				(font
@@
 		)
 		(property "Description" "Unpolarized capacitor"
-			(at 182.88 139.7 0)
+			(at 171.45 139.7 0)
 			(effects
 				(font
@@
 		)
 		(property "Mouser Part Number" "81-GRT188R61H225KE3D"
-			(at 182.88 139.7 0)
+			(at 171.45 139.7 0)
 			(effects
 				(font
@@
 	(symbol
 		(lib_id "power:GND")
-		(at 182.88 144.78 0)
+		(at 171.45 144.78 0)
 		(unit 1)
 		(exclude_from_sim no)
@@
 		(fields_autoplaced yes)
 		(property "Reference" "#PWR0204"
-			(at 182.88 151.13 0)
+			(at 171.45 151.13 0)
 			(effects
 				(font
@@
 		)
 		(property "Value" "GND"
-			(at 182.88 149.86 0)
+			(at 171.45 149.86 0)
 			(effects
 				(font
@@
 		)
 		(property "Footprint" ""
-			(at 182.88 144.78 0)
+			(at 171.45 144.78 0)
 			(effects
 				(font
@@
 		)
 		(property "Datasheet" ""
-			(at 182.88 144.78 0)
+			(at 171.45 144.78 0)
 			(effects
 				(font
@@
 		)
 		(property "Description" "Power symbol creates a global label with name \"GND\" , ground"
-			(at 182.88 144.78 0)
+			(at 171.45 144.78 0)
 			(effects
 				(font
@@
 	)
 	(symbol
+		(lib_id "Device:C")
+		(at 184.15 138.43 0)
+		(mirror x)
+		(unit 1)
+		(exclude_from_sim no)
+		(in_bom yes)
+		(on_board yes)
+		(dnp no)
+		(property "Reference" "C209"
+			(at 176.53 138.43 90)
+			(effects
+				(font
+					(size 1.27 1.27)
+				)
+			)
+		)
+		(property "Value" "100n"
+			(at 179.07 138.43 90)
+			(effects
+				(font
+					(size 1.27 1.27)
+				)
+			)
+		)
+		(property "Footprint" "Capacitor_SMD:C_0402_1005Metric"
+			(at 185.1152 134.62 0)
+			(effects
+				(font
+					(size 1.27 1.27)
+				)
+				(hide yes)
+			)
+		)
+		(property "Datasheet" "~"
+			(at 184.15 138.43 0)
+			(effects
+				(font
+					(size 1.27 1.27)
+				)
+				(hide yes)
+			)
+		)
+		(property "Description" "Unpolarized capacitor"
+			(at 184.15 138.43 0)
+			(effects
+				(font
+					(size 1.27 1.27)
+				)
+				(hide yes)
+			)
+		)
+		(property "Mouser Part Number" "81-GRM155R62A104KE4D"
+			(at 184.15 138.43 90)
+			(effects
+				(font
+					(size 1.27 1.27)
+				)
+				(hide yes)
+			)
+		)
+		(pin "2"
+		)
+		(pin "1"
+		)
+		(instances
+			(project "STEVEannouncer"
+				(path "/1a37937a-d840-40ca-a420-44780efca6fe/eebf1098-e67c-4d58-86f4-2b87a99f6ef8"
+					(reference "C209")
+					(unit 1)
+				)
+			)
+		)
+	)
+	(symbol
 		(lib_id "power:GND")
 		(at 234.95 137.16 90)
@@
 					(unit 1)
 				)
+			)
+		)
+	)
+	(symbol
+		(lib_id "power:-5V")
+		(at 184.15 142.24 180)
+		(unit 1)
+		(exclude_from_sim no)
+		(in_bom yes)
+		(on_board yes)
+		(dnp no)
+		(fields_autoplaced yes)
+		(property "Reference" "#PWR0213"
+			(at 184.15 138.43 0)
+			(effects
+				(font
+					(size 1.27 1.27)
+				)
+				(hide yes)
+			)
+		)
+		(property "Value" "-5V"
+			(at 184.15 147.32 0)
+			(effects
+				(font
+					(size 1.27 1.27)
+				)
+			)
+		)
+		(property "Footprint" ""
+			(at 184.15 142.24 0)
+			(effects
+				(font
+					(size 1.27 1.27)
+				)
+				(hide yes)
+			)
+		)
+		(property "Datasheet" ""
+			(at 184.15 142.24 0)
+			(effects
+				(font
+					(size 1.27 1.27)
+				)
+				(hide yes)
+			)
+		)
+		(property "Description" "Power symbol creates a global label with name \"-5V\""
+			(at 184.15 142.24 0)
+			(effects
+				(font
+					(size 1.27 1.27)
+				)
+				(hide yes)
+			)
+		)
+		(pin "1"
+		)
+		(instances
+			(project "STEVEannouncer"
+				(path "/1a37937a-d840-40ca-a420-44780efca6fe/eebf1098-e67c-4d58-86f4-2b87a99f6ef8"
+					(reference "#PWR0213")
+					(unit 1)
+				)

Commit message: Yeet
Parts:
- added D204: LED, LED_SMD:LED_0603_1608Metric, symbol Device:LED
- added R209: 1k, Resistor_SMD:R_0402_1005Metric, symbol Device:R
Connections:
- net +5V: now also R209.1
- net GND: now also D204.1 (K)
- new net: D204.2 (A), R209.2

Commit message: I think I can fab this????
Parts:
- U201, U202: footprint Package_TO_SOT_SMD:SOT-23-6 -> STEVEannouncer:SOT-23-6
Changed lines of the file:
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@@
 			)
 		)
-		(property "Footprint" "Package_TO_SOT_SMD:SOT-23-6"
+		(property "Footprint" "STEVEannouncer:SOT-23-6"
 			(at 201.93 137.16 0)
 			(effects
@@
 			)
 		)
-		(property "Footprint" "Package_TO_SOT_SMD:SOT-23-6"
+		(property "Footprint" "STEVEannouncer:SOT-23-6"
 			(at 201.93 104.14 0)
 			(effects

Commit message: Enclosure files
Parts:
- D204: Mouser Part Number (none) -> 859-LTST-C191KRKT
- R201: Mouser Part Number (none) -> 603-RC0402FR-7W1ML
- R202: Mouser Part Number (none) -> 603-RC0402FR-13330KL
- R203, R205, R206: Mouser Part Number (none) -> 603-RC0402FR-1320KL
- R204: Mouser Part Number (none) -> 652-CR1206-JW-100ELF
- R207, R208: Mouser Part Number (none) -> 652-CR0402-FX8062GLF
- R209: Mouser Part Number (none) -> 708-RMCF0402FT1K00
Changed lines of the file:
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@@
+			)
+		)
+		(property "Mouser Part Number" "603-RC0402FR-1320KL"
+			(at 212.09 111.76 0)
+			(effects
+				(font
+					(size 1.27 1.27)
+				)
+				(hide yes)
 			)
 		)
@@
 			)
 		)
+		(property "Mouser Part Number" "603-RC0402FR-1320KL"
+			(at 212.09 144.78 0)
+			(effects
+				(font
+					(size 1.27 1.27)
+				)
+				(hide yes)
+			)
+		)
 		(pin "1"
 		)
@@
 			)
 		)
+		(property "Mouser Part Number" "603-RC0402FR-1320KL"
+			(at 74.93 67.31 0)
+			(effects
+				(font
+					(size 1.27 1.27)
+				)
+				(hide yes)
+			)
+		)
 		(pin "1"
 		)
@@
 			)
 		)
+		(property "Mouser Part Number" "708-RMCF0402FT1K00"
+			(at 144.78 67.31 90)
+			(effects
+				(font
+					(size 1.27 1.27)
+				)
+				(hide yes)
+			)
+		)
 		(pin "1"
 		)
@@
 			)
 		)
+		(property "Mouser Part Number" "652-CR0402-FX8062GLF"
+			(at 220.98 139.7 90)
+			(effects
+				(font
+					(size 1.27 1.27)
+				)
+				(hide yes)
+			)
+		)
 		(pin "1"
 		)
@@
 			)
 		)
+		(property "Mouser Part Number" "603-RC0402FR-7W1ML"
+			(at 58.42 63.5 0)
+			(effects
+				(font
+					(size 1.27 1.27)
+				)
+				(hide yes)
+			)
+		)
 		(pin "1"
 		)
@@
 			)
 		)
+		(property "Mouser Part Number" "859-LTST-C191KRKT"
+			(at 154.94 67.31 0)
+			(effects
+				(font
+					(size 1.27 1.27)
+				)
+				(hide yes)
+			)
+		)
 		(pin "1"
 		)
@@
 			)
 		)
+		(property "Mouser Part Number" "652-CR1206-JW-100ELF"
+			(at 101.6 93.98 0)
+			(effects
+				(font
+					(size 1.27 1.27)
+				)
+				(hide yes)
+			)
+		)
 		(pin "1"
 		)
@@
 			)
 		)
+		(property "Mouser Part Number" "603-RC0402FR-13330KL"
+			(at 58.42 87.63 0)
+			(effects
+				(font
+					(size 1.27 1.27)
+				)
+				(hide yes)
+			)
+		)
 		(pin "1"
 		)
@@
 			(effects
 				(font
+					(size 1.27 1.27)
+				)
+				(hide yes)
+			)
+		)
+		(property "Mouser Part Number" "652-CR0402-FX8062GLF"
+			(at 220.98 106.68 90)
+			(effects
+				(font
