File: PCB/Power.kicad_sch (KiCad schematic)
At the start: 29 parts, among them J201 Barrel_Jack_Switch, Q201 BC847, Q202 BCV49, U201 LV3842, U202 LV3842

Commit message: revisionnnnn
Parts:
- added R210: 80.6k, Resistor_SMD:R_0402_1005Metric, symbol Device:R
- added R211: 10k, Resistor_SMD:R_0402_1005Metric, symbol Device:R
Connections:
- net +5V: now also U202.4 (EN)
- net GND: now also R211.1
- net vbulk: now also R210.2; no longer U201.4 (EN), U202.4 (EN)
- new net: R210.1, R211.2, U201.4 (EN)
Other:
- moved on the sheet: C203
