File: PCB/Power.kicad_sch (KiCad schematic)
At the start: 31 parts, among them J201 Barrel_Jack_Switch, Q201 BC847, Q202 BCV49, U201 LV3842, U202 LV3842

Commit message: Rev 2025-07-20
Parts:
- D201: Gearlabs Part Number D-Zener-5V6-123-2 -> (none)
- Q202: footprint Package_TO_SOT_SMD:SOT-89-3 -> STEVEannouncer:SOT-89-3; symbol Device:Q_NPN_Darlington -> Transistor_BJT:Q_NPN_Darlington_BCE
- R210: Mouser Part Number (none) -> 652-CR0402-FX8062GLF
- R211: Mouser Part Number (none) -> 652-CR0402FX-1002GLF
Connections:
- net Darl_B: now reaches C201.1, Q201.3 (C), R201.2, R202.1, R203.2
- net Darl_B: now also Q202.1 (B); no longer Q202.3 (B)
- net Pin2_Bulk: now reaches C201.2, D202.2 (A), Q201.2 (E), R202.2, R204.2
- net Darl_E: now reaches Q201.1 (B), R204.1
- net Darl_E: now also Q202.3 (E); no longer Q202.1 (E)
Changed lines of the file:
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@@
 		)
 	)
+	(label "Darl_E"
+		(at 101.6 85.09 90)
+		(effects
+			(font
+				(size 1.27 1.27)
+			)
+			(justify left bottom)
+		)
+	)
+	(label "Pin2_Bulk"
+		(at 80.01 101.6 0)
+		(effects
+			(font
+				(size 1.27 1.27)
+			)
+			(justify left bottom)
+		)
+	)
 	(label "vbulk"
 		(at 152.4 101.6 0)
@@
 		)
 	)
+	(label "Darl_B"
+		(at 80.01 73.66 0)
+		(effects
+			(font
+				(size 1.27 1.27)
+			)
+			(justify left bottom)
+		)
+	)
 	(global_label "IFB_PIN2"
 		(shape input)
@@
 			)
 		)
-		(property "Mouser Part#" ""
-			(at 74.93 57.15 0)
-			(effects
-				(font
-					(size 1.27 1.27)
-				)
-				(hide yes)
-			)
-		)
-		(property "Gearlabs Part Number" "D-Zener-5V6-123-2"
-			(at 74.93 57.15 0)
-			(effects
-				(font
-					(size 1.27 1.27)
-				)
-				(hide yes)
-			)
-		)
 		(pin "2"
 		)
@@
 			)
 		)
-		(property "Sim.Pins" "1=K 2=A"
-			(at 154.94 67.31 0)
-			(effects
-				(font
-					(size 1.27 1.27)
-				)
-				(hide yes)
-			)
-		)
 		(property "Mouser Part Number" "859-LTST-C191KRKT"
 			(at 154.94 67.31 0)
@@
 	)
 	(symbol
-		(lib_id "Device:Q_NPN_Darlington")
+		(lib_id "Transistor_BJT:Q_NPN_Darlington_BCE")
 		(at 99.06 73.66 0)
 		(unit 1)
@@
 			)
 		)
-		(property "Footprint" "Package_TO_SOT_SMD:SOT-89-3"
+		(property "Footprint" "STEVEannouncer:SOT-89-3"
 			(at 104.14 71.12 0)
 			(effects
@@
 			)
 		)
-		(property "Datasheet" "~"
+		(property "Datasheet" ""
 			(at 99.06 73.66 0)
 			(effects
@@
 			)
 		)
-		(property "Description" "NPN Darlington  bipolar junction transistor"
+		(property "Description" ""
 			(at 99.06 73.66 0)
 			(effects
@@
 			)
 		)
+		(property "Mouser Part Number" "652-CR0402-FX8062GLF"
+			(at 182.88 106.68 90)
+			(effects
+				(font
+					(size 1.27 1.27)
+				)
+				(hide yes)
+			)
+		)
 		(pin "1"
 		)
@@
 			(at 182.88 116.84 0)
 			(effects
+				(font
+					(size 1.27 1.27)
+				)
+				(hide yes)
+			)
+		)
+		(property "Mouser Part Number" "652-CR0402FX-1002GLF"
+			(at 182.88 116.84 0)
+			(effects

Commit message: Tidying up
Parts:
- U201, U202: footprint STEVEannouncer:SOT-23-6 -> Package_TO_SOT_SMD:SOT-23-6
Connections:
- net Darl_B: now also Q201.C; no longer Q201.3 (C)
- net Darl_E: now also Q201.B; no longer Q201.1 (B)
- net Pin2_Bulk: now also Q201.E; no longer Q201.2 (E)
- net at L202.1, U202.6 (SW): now also C206.1; no longer C206.2
- net at U202.1 (Boot): now also C206.2; no longer C206.1
- net at U201.1 (Boot): now also C205.2; no longer C205.1
- net at L201.1, U201.6 (SW): now also C205.1; no longer C205.2
Other:
- note added: "+5V Rail"
- note added: "-5V Rail"
- note added: "DC Input"
- note added: "Phantom Power Input"
- note added: "Power Light"
- moved on the sheet: C203, C204, C205, C206, C207, C208, D203, J201, L201, L202, R205, R206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
